Commit message: single arm config

File: cr5_dual_description/urdf/cr5_dual.urdf (robot description, URDF)
Before this commit: robot fiveages_cr5_dual_station, 18 links, 17 joints
Links:
- link left_Link6: geometry collision box size=0.08 0.08 0.14; collision box size=0.18 0.04 0.04
- link right_Link6: geometry collision box size=0.08 0.08 0.14; collision box size=0.18 0.04 0.04
Joints:
- joint left_joint4: limit lower=-6.283185307179586 upper=6.283185307179586 effort=300 velocity=3.141592653589793 -> lower=-6.283185307179586 upper=2.2591366109921265 effort=300 velocity=3.141592653589793
- joint left_tcp_joint: origin xyz=0 0 0.29 -> xyz=0 0 0.21
- joint right_tcp_joint: origin xyz=0 0 0.29 -> xyz=0 0 0.21

File: cr5_dual_description/xacro/grippers.xacro (robot description, xacro)
@@ -31,5 +31,35 @@
     </joint>
   </xacro:if>
-  <xacro:if value="${'$(arg type)' == 'AG2F90-Ct'}">
+  <xacro:if value="${'$(arg type)' == 'AG2F90-C'}">
+    <xacro:include filename="$(find changingtek_description)/xacro/AG2F90-C.xacro"/>
+    <xacro:AG2F90-C name="left" use_flange="true"/>
+    <xacro:AG2F90-C name="right" use_flange="true"/>
+    <joint name="left_gripper_fixed" type="fixed">
+      <parent link="left_Link6"/>
+      <child link="left_flange"/>
+      <origin rpy="0 0 ${PI/2}"/>
+    </joint>
+    <joint name="right_gripper_fixed" type="fixed">
+      <parent link="right_Link6"/>
+      <child link="right_flange"/>
+      <origin rpy="0 0 ${PI/2}"/>
+    </joint>
+  </xacro:if>
+  <xacro:if value="${'$(arg type)' == 'left_arm'}">
+    <xacro:include filename="$(find changingtek_description)/xacro/AG2F90-C.xacro"/>
+    <xacro:AG2F90-C name="left" use_flange="true"/>
+    <xacro:AG2F90-C name="right" use_flange="true"/>
+    <joint name="left_gripper_fixed" type="fixed">
+      <parent link="left_Link6"/>
+      <child link="left_flange"/>
+      <origin rpy="0 0 ${PI/2}"/>
+    </joint>
+    <joint name="right_gripper_fixed" type="fixed">
+      <parent link="right_Link6"/>
+      <child link="right_flange"/>
+      <origin rpy="0 0 ${PI/2}"/>
+    </joint>
+  </xacro:if>
+  <xacro:if value="${'$(arg type)' == 'right_arm'}">
     <xacro:include filename="$(find changingtek_description)/xacro/AG2F90-C.xacro"/>
     <xacro:AG2F90-C name="left" use_flange="true"/>
