Commit message: add cartesion motion controller

File: cr5_dual_description/urdf/cr5_dual_left_arm.urdf (robot description, URDF)
Before this commit: robot fiveages_cr5_dual_station, 18 links, 17 joints
Joints:
- joint left_joint4: limit lower=-6.283185307179586 upper=6.283185307179586 effort=300 velocity=3.141592653589793 -> lower=-6.283185307179586 upper=2.2591366109921265 effort=300 velocity=3.141592653589793

File: cr5_dual_description/xacro/ros2_control/robot.xacro (robot description, xacro)
@@ -147,5 +147,5 @@
             <xacro:cr5_interfaces name="right"/>
             <!-- 夹爪接口 - 参考CR5的模块化设计 -->
-            <xacro:if value="${'$(arg type)' == 'AG2F90-C' or '$(arg type)' == 'AG2F90-C-Soft'}">
+            <xacro:if value="${'$(arg type)' == 'AG2F90-C' or '$(arg type)' == 'AG2F90-C-Soft'  or '$(arg type)' == 'left_arm'}">
                 <xacro:include filename="$(find changingtek_description)/xacro/ros2_control/AG2F90-C.xacro"/>
                 <xacro:ag2f90c_interfaces name="left"/>
