Commit message: dual arm for isaac sim

File: cr5_dual_description/xacro/grippers.xacro (robot description, xacro)
@@ -31,3 +31,18 @@
     </joint>
   </xacro:if>
+  <xacro:if value="${'$(arg type)' == 'AG2F90-Ct'}">
+    <xacro:include filename="$(find changingtek_description)/xacro/AG2F90-C.xacro"/>
+    <xacro:AG2F90-C name="left" use_flange="true"/>
+    <xacro:AG2F90-C name="right" use_flange="true"/>
+    <joint name="left_gripper_fixed" type="fixed">
+      <parent link="left_Link6"/>
+      <child link="left_flange"/>
+      <origin rpy="0 0 ${PI/2}"/>
+    </joint>
+    <joint name="right_gripper_fixed" type="fixed">
+      <parent link="right_Link6"/>
+      <child link="right_flange"/>
+      <origin rpy="0 0 ${PI/2}"/>
+    </joint>
+  </xacro:if>
 </robot>

File: cr5_dual_description/xacro/robot.xacro (robot description, xacro)
@@ -1,4 +1,4 @@
 <?xml version="1.0"?>
-<robot name="fiveages_cr5_dual_station" xmlns:xacro="http://www.ros.org/wiki/xacro">
+<robot name="DobotCR5_Dual" xmlns:xacro="http://www.ros.org/wiki/xacro">
   <xacro:arg name="collider" default="convex"/>
   <link name="base_link">

File: cr5_dual_description/xacro/ros2_control/robot.xacro (robot description, xacro)
@@ -21,5 +21,5 @@
             </hardware>
             <xacro:cr5_interfaces name="left"/>
-            <xacro:if value="${'$(arg type)' == 'AG2F90-C-Soft'}">
+            <xacro:if value="${'$(arg type)' != 'empty'}">
                 <joint name="left_gripper_joint">
                     <command_interface name="position"/>
@@ -40,5 +40,5 @@
             </hardware>
             <xacro:cr5_interfaces name="right"/>
-            <xacro:if value="${'$(arg type)' == 'AG2F90-C-Soft'}">
+            <xacro:if value="${'$(arg type)' != 'empty'}">
                 <joint name="right_gripper_joint">
                     <command_interface name="position"/>
@@ -50,19 +50,50 @@
         </ros2_control>
     </xacro:if>
-    <xacro:unless value="${'$(arg ros2_control_hardware_type)' == 'real'}">
-        <!-- Unified ros2_control system -->
+    <xacro:if value="${'$(arg ros2_control_hardware_type)' == 'isaac'}">
+        <!-- Isaac Sim: Use two separate topic_based systems for left and right arms -->
+        <ros2_control name="cr5_left_system" type="system">
+            <hardware>
+                <plugin>topic_based_ros2_control/TopicBasedSystem</plugin>
+                <param name="joint_commands_topic">/isaac_left/joint_command</param>
+                <param name="joint_states_topic">/isaac_left/joint_states</param>
+                <param name="joint_name_prefix">left_</param>
+            </hardware>
+            <!-- 左臂接口 -->
+            <xacro:cr5_interfaces name="left"/>
+            <!-- 左臂夹爪接口 -->
+            <xacro:if value="${'$(arg type)' == 'AG2F90-C' or '$(arg type)' == 'AG2F90-C-Soft'}">
+                <xacro:include filename="$(find changingtek_description)/xacro/ros2_control/AG2F90-C.xacro"/>
+                <xacro:ag2f90c_interfaces name="left"/>
+            </xacro:if>
+            <xacro:if value="${'$(arg type)' == 'robotiq85'}">
+                <xacro:include filename="$(find robotiq_description)/xacro/ros2_control/2F85.xacro"/>
+                <xacro:robotiq_2f85_interfaces name="left"/>
+            </xacro:if>
+        </ros2_control>
+        <ros2_control name="cr5_right_system" type="system">
+            <hardware>
+                <plugin>topic_based_ros2_control/TopicBasedSystem</plugin>
+                <param name="joint_commands_topic">/isaac_right/joint_command</param>
+                <param name="joint_states_topic">/isaac_right/joint_states</param>
+                <param name="joint_name_prefix">right_</param>
+            </hardware>
+            <!-- 右臂接口 -->
+            <xacro:cr5_interfaces name="right"/>
+            <!-- 右臂夹爪接口 -->
+            <xacro:if value="${'$(arg type)' == 'AG2F90-C' or '$(arg type)' == 'AG2F90-C-Soft'}">
+                <xacro:include filename="$(find changingtek_description)/xacro/ros2_control/AG2F90-C.xacro"/>
+                <xacro:ag2f90c_interfaces name="right"/>
+            </xacro:if>
+            <xacro:if value="${'$(arg type)' == 'robotiq85'}">
+                <xacro:include filename="$(find robotiq_description)/xacro/ros2_control/2F85.xacro"/>
+                <xacro:robotiq_2f85_interfaces name="right"/>
+            </xacro:if>
+        </ros2_control>
+    </xacro:if>
+    <xacro:if value="${'$(arg ros2_control_hardware_type)' == 'gz'}">
+        <!-- Gazebo Simulator: Unified ros2_control system -->
         <ros2_control name="cr5_dual_system" type="system">
             <hardware>
-                <xacro:if value="${'$(arg ros2_control_hardware_type)' == 'gz'}">
-                    <plugin>gz_ros2_control/GazeboSimSystem</plugin>
-                </xacro:if>
-                <xacro:if value="${'$(arg ros2_control_hardware_type)' == 'mock_components'}">
-                    <plugin>mock_components/GenericSystem</plugin>
-                </xacro:if>
-                <xacro:if value="${'$(arg ros2_control_hardware_type)' == 'isaac'}">
-                    <plugin>topic_based_ros2_control/TopicBasedSystem</plugin>
-                    <param name="joint_commands_topic">/isaac/joint_command</param>
-                    <param name="joint_states_topic">/isaac/joint_states</param>
-                </xacro:if>
+                <plugin>gz_ros2_control/GazeboSimSystem</plugin>
             </hardware>
             <!-- 左臂接口 -->
@@ -91,4 +122,27 @@
             <!-- Gazebo configuration for CR5 dual arm -->
         </xacro:if>
-    </xacro:unless>
+    </xacro:if>
+    <xacro:if value="${'$(arg ros2_control_hardware_type)' == 'mock_components'}">
+        <!-- Mock Components: Unified ros2_control system -->
+        <ros2_control name="cr5_dual_system" type="system">
+            <hardware>
+                <plugin>mock_components/GenericSystem</plugin>
+            </hardware>
+            <!-- 左臂接口 -->
+            <xacro:cr5_interfaces name="left"/>
+            <!-- 右臂接口 -->
+            <xacro:cr5_interfaces name="right"/>
+            <!-- 夹爪接口 - 参考CR5的模块化设计 -->
+            <xacro:if value="${'$(arg type)' == 'AG2F90-C' or '$(arg type)' == 'AG2F90-C-Soft'}">
+                <xacro:include filename="$(find changingtek_description)/xacro/ros2_control/AG2F90-C.xacro"/>
+                <xacro:ag2f90c_interfaces name="left"/>
+                <xacro:ag2f90c_interfaces name="right"/>
+            </xacro:if>
+            <xacro:if value="${'$(arg type)' == 'robotiq85'}">
+                <xacro:include filename="$(find robotiq_description)/xacro/ros2_control/2F85.xacro"/>
+                <xacro:robotiq_2f85_interfaces name="left"/>
+                <xacro:robotiq_2f85_interfaces name="right"/>
+            </xacro:if>
+        </ros2_control>
+    </xacro:if>
 </robot>

Commit message: 给cr5_dual增加AG2F120S夹爪的相关配置

File: cr5_dual_description/xacro/grippers.xacro (robot description, xacro)
@@ -46,3 +46,16 @@
     </joint>
   </xacro:if>
+  <xacro:if value="${'$(arg type)' == 'AG2F120S'}">
+    <xacro:include filename="$(find changingtek_description)/xacro/AG2F120S.xacro"/>
+    <xacro:AG2F120S name="left"/>
+    <xacro:AG2F120S name="right"/>
+    <joint name="left_gripper_fix" type="fixed">
+      <parent link="left_Link6"/>
+      <child link="left_gripper_base"/>
+    </joint>
+    <joint name="right_gripper_fix" type="fixed">
+      <parent link="right_Link6"/>
+      <child link="right_gripper_base"/>
+    </joint>
+  </xacro:if>
 </robot>

File: cr5_dual_description/xacro/ros2_control/robot.xacro (robot description, xacro)
@@ -70,4 +70,8 @@
                 <xacro:robotiq_2f85_interfaces name="left"/>
             </xacro:if>
+            <xacro:if value="${'$(arg type)' == 'AG2F120S'}">
+                <xacro:include filename="$(find changingtek_description)/xacro/ros2_control/AG2F120S.xacro"/>
+                <xacro:ag2f120s_interfaces name="left"/>
+            </xacro:if>
         </ros2_control>
         <ros2_control name="cr5_right_system" type="system">
@@ -88,4 +92,8 @@
                 <xacro:include filename="$(find robotiq_description)/xacro/ros2_control/2F85.xacro"/>
                 <xacro:robotiq_2f85_interfaces name="right"/>
+            </xacro:if>
+            <xacro:if value="${'$(arg type)' == 'AG2F120S'}">
+                <xacro:include filename="$(find changingtek_description)/xacro/ros2_control/AG2F120S.xacro"/>
+                <xacro:ag2f120s_interfaces name="right"/>
             </xacro:if>
         </ros2_control>
@@ -111,4 +119,9 @@
                 <xacro:robotiq_2f85_interfaces name="left"/>
                 <xacro:robotiq_2f85_interfaces name="right"/>
+            </xacro:if>
+            <xacro:if value="${'$(arg type)' == 'AG2F120S'}">
+                <xacro:include filename="$(find changingtek_description)/xacro/ros2_control/AG2F120S.xacro"/>
+                <xacro:ag2f120s_interfaces name="left"/>
+                <xacro:ag2f120s_interfaces name="right"/>
             </xacro:if>
         </ros2_control>
@@ -144,4 +157,9 @@
                 <xacro:robotiq_2f85_interfaces name="right"/>
             </xacro:if>
+            <xacro:if value="${'$(arg type)' == 'AG2F120S'}">
+                <xacro:include filename="$(find changingtek_description)/xacro/ros2_control/AG2F120S.xacro"/>
+                <xacro:ag2f120s_interfaces name="left"/>
+                <xacro:ag2f120s_interfaces name="right"/>
+            </xacro:if>
         </ros2_control>
     </xacro:if>

Commit message: Remove LFS tracking configuration

File: cr5_dual_description/xacro/grippers.xacro (robot description, xacro)
@@ -46,16 +46,3 @@
     </joint>
   </xacro:if>
-  <xacro:if value="${'$(arg type)' == 'AG2F120S'}">
-    <xacro:include filename="$(find changingtek_description)/xacro/AG2F120S.xacro"/>
-    <xacro:AG2F120S name="left"/>
-    <xacro:AG2F120S name="right"/>
-    <joint name="left_gripper_fix" type="fixed">
-      <parent link="left_Link6"/>
-      <child link="left_gripper_base"/>
-    </joint>
-    <joint name="right_gripper_fix" type="fixed">
-      <parent link="right_Link6"/>
-      <child link="right_gripper_base"/>
-    </joint>
-  </xacro:if>
 </robot>

File: cr5_dual_description/xacro/ros2_control/robot.xacro (robot description, xacro)
@@ -70,8 +70,4 @@
                 <xacro:robotiq_2f85_interfaces name="left"/>
             </xacro:if>
-            <xacro:if value="${'$(arg type)' == 'AG2F120S'}">
-                <xacro:include filename="$(find changingtek_description)/xacro/ros2_control/AG2F120S.xacro"/>
-                <xacro:ag2f120s_interfaces name="left"/>
-            </xacro:if>
         </ros2_control>
         <ros2_control name="cr5_right_system" type="system">
@@ -92,8 +88,4 @@
                 <xacro:include filename="$(find robotiq_description)/xacro/ros2_control/2F85.xacro"/>
                 <xacro:robotiq_2f85_interfaces name="right"/>
-            </xacro:if>
-            <xacro:if value="${'$(arg type)' == 'AG2F120S'}">
-                <xacro:include filename="$(find changingtek_description)/xacro/ros2_control/AG2F120S.xacro"/>
-                <xacro:ag2f120s_interfaces name="right"/>
             </xacro:if>
         </ros2_control>
@@ -119,9 +111,4 @@
                 <xacro:robotiq_2f85_interfaces name="left"/>
                 <xacro:robotiq_2f85_interfaces name="right"/>
-            </xacro:if>
-            <xacro:if value="${'$(arg type)' == 'AG2F120S'}">
-                <xacro:include filename="$(find changingtek_description)/xacro/ros2_control/AG2F120S.xacro"/>
-                <xacro:ag2f120s_interfaces name="left"/>
-                <xacro:ag2f120s_interfaces name="right"/>
             </xacro:if>
         </ros2_control>
@@ -157,9 +144,4 @@
                 <xacro:robotiq_2f85_interfaces name="right"/>
             </xacro:if>
-            <xacro:if value="${'$(arg type)' == 'AG2F120S'}">
-                <xacro:include filename="$(find changingtek_description)/xacro/ros2_control/AG2F120S.xacro"/>
-                <xacro:ag2f120s_interfaces name="left"/>
-                <xacro:ag2f120s_interfaces name="right"/>
-            </xacro:if>
         </ros2_control>
     </xacro:if>
