Commit message: modified ocs2 config

File: cr5_description/urdf/cr5.urdf (robot description, URDF)
Before this commit: robot DobotCR5, 8 links, 7 joints
Links:
- link Link6: geometry collision box size=0.06 0.04 0.14; collision cylinder length=0.138392 radius=0.041707
- link base_link: geometry collision box size=1.5 1.5 0.05; visual mesh filename=package://cr5_description/meshes/visual/base_link.obj
