Commit message: fix dual isaac sim

File: cr5_description/xacro/grippers.xacro (robot description, xacro)
@@ -28,4 +28,10 @@
 			<origin rpy="0 0 ${PI/2}"/>
 		</joint>
+		<link name="hand_camera"/>
+		<joint name="hand_camera_joint" type="fixed">
+			<parent link="Link6"/>
+			<child link="hand_camera"/>
+			<origin xyz="-0.0232323851 -0.0658349999 0.1368881312" rpy="-0.1206332889 0.0085965555 0.0669556163"/>
+		</joint>
 	</xacro:if>
 	<xacro:if value="${'$(arg type)' == 'AG2F120S'}">

File: cr5_dual_description/xacro/robot.xacro (robot description, xacro)
@@ -2,4 +2,5 @@
 <robot name="DobotCR5_Dual" xmlns:xacro="http://www.ros.org/wiki/xacro">
   <xacro:arg name="collider" default="convex"/>
+  <xacro:property name="tf_params" value="${xacro.load_yaml('$(find cr5_description)/xacro/tf_params.yaml')['tf_params']}"/>
   <link name="base_link">
     <visual>
@@ -15,6 +16,6 @@
   </link>
   <xacro:include filename="$(find cr5_description)/xacro/arm.xacro"/>
-  <xacro:CR5 name="left" collider="$(arg collider)"/>
-  <xacro:CR5 name="right" collider="$(arg collider)"/>
+  <xacro:CR5 name="left" collider="$(arg collider)" tf_params="${tf_params}"/>
+  <xacro:CR5 name="right" collider="$(arg collider)" tf_params="${tf_params}"/>
   <!-- Initial guess; measure or adjust in RViz for final mounting pose -->
   <joint name="left_arm_mount" type="fixed">

File: cr5_dual_description/xacro/ros2_control/robot.xacro (robot description, xacro)
@@ -1,148 +1,134 @@
 <?xml version="1.0" ?>
 <robot name="fiveages_cr5_dual_station" xmlns:xacro="http://www.ros.org/wiki/xacro">
-    <link name="world"/>
-    <joint name="world_fixed" type="fixed">
-        <parent link="world"/>
-        <child link="base_link"/>
-        <origin/>
-    </joint>
-    <!-- Include the base robot structure -->
-    <xacro:include filename="$(find cr5_dual_description)/xacro/robot.xacro"/>
-    <xacro:include filename="$(find cr5_description)/xacro/ros2_control/interfaces.xacro"/>
-    <xacro:if value="${'$(arg ros2_control_hardware_type)' == 'real'}">
-        <ros2_control name="cr5_left_system" type="system">
-            <hardware>
-                <plugin>dobot_ros2_control/DobotHardware</plugin>
-                <param name="robot_ip">192.168.5.33</param>
-                <param name="gain">200</param>
-                <param name="aheadtime">20</param>
-                <param name="speed_factor">100</param>
-                <param name="servo_time">0.3</param>
-            </hardware>
-            <xacro:cr5_interfaces name="left"/>
-            <xacro:if value="${'$(arg type)' != 'empty'}">
-                <joint name="left_gripper_joint">
-                    <command_interface name="position"/>
-                    <state_interface name="position">
-                        <param name="initial_value">0</param>
-                    </state_interface>
-                </joint>
-            </xacro:if>
-        </ros2_control>
-        <ros2_control name="cr5_right_system" type="system">
-            <hardware>
-                <plugin>dobot_ros2_control/DobotHardware</plugin>
-                <param name="robot_ip">192.168.5.34</param>
-                <param name="gain">200</param>
-                <param name="aheadtime">20</param>
-                <param name="speed_factor">100</param>
-                <param name="servo_time">0.3</param>
-            </hardware>
-            <xacro:cr5_interfaces name="right"/>
-            <xacro:if value="${'$(arg type)' != 'empty'}">
-                <joint name="right_gripper_joint">
-                    <command_interface name="position"/>
-                    <state_interface name="position">
-                        <param name="initial_value">0</param>
-                    </state_interface>
-                </joint>
-            </xacro:if>
-        </ros2_control>
-    </xacro:if>
-    <xacro:if value="${'$(arg ros2_control_hardware_type)' == 'isaac'}">
-        <!-- Isaac Sim: Use two separate topic_based systems for left and right arms -->
-        <ros2_control name="cr5_left_system" type="system">
-            <hardware>
-                <plugin>topic_based_ros2_control/TopicBasedSystem</plugin>
-                <param name="joint_commands_topic">/isaac_left/joint_command</param>
-                <param name="joint_states_topic">/isaac_left/joint_states</param>
-                <param name="joint_name_prefix">left_</param>
-            </hardware>
-            <!-- 左臂接口 -->
-            <xacro:cr5_interfaces name="left"/>
-            <!-- 左臂夹爪接口 -->
-            <xacro:if value="${'$(arg type)' == 'AG2F90-C' or '$(arg type)' == 'AG2F90-C-Soft'}">
-                <xacro:include filename="$(find changingtek_description)/xacro/ros2_control/AG2F90-C.xacro"/>
-                <xacro:ag2f90c_interfaces name="left"/>
-            </xacro:if>
-            <xacro:if value="${'$(arg type)' == 'robotiq85'}">
-                <xacro:include filename="$(find robotiq_description)/xacro/ros2_control/2F85.xacro"/>
-                <xacro:robotiq_2f85_interfaces name="left"/>
-            </xacro:if>
-        </ros2_control>
-        <ros2_control name="cr5_right_system" type="system">
-            <hardware>
-                <plugin>topic_based_ros2_control/TopicBasedSystem</plugin>
-                <param name="joint_commands_topic">/isaac_right/joint_command</param>
-                <param name="joint_states_topic">/isaac_right/joint_states</param>
-                <param name="joint_name_prefix">right_</param>
-            </hardware>
-            <!-- 右臂接口 -->
-            <xacro:cr5_interfaces name="right"/>
-            <!-- 右臂夹爪接口 -->
-            <xacro:if value="${'$(arg type)' == 'AG2F90-C' or '$(arg type)' == 'AG2F90-C-Soft'}">
-                <xacro:include filename="$(find changingtek_description)/xacro/ros2_control/AG2F90-C.xacro"/>
-                <xacro:ag2f90c_interfaces name="right"/>
-            </xacro:if>
-            <xacro:if value="${'$(arg type)' == 'robotiq85'}">
-                <xacro:include filename="$(find robotiq_description)/xacro/ros2_control/2F85.xacro"/>
-                <xacro:robotiq_2f85_interfaces name="right"/>
-            </xacro:if>
-        </ros2_control>
-    </xacro:if>
-    <xacro:if value="${'$(arg ros2_control_hardware_type)' == 'gz'}">
-        <!-- Gazebo Simulator: Unified ros2_control system -->
-        <ros2_control name="cr5_dual_system" type="system">
-            <hardware>
-                <plugin>gz_ros2_control/GazeboSimSystem</plugin>
-            </hardware>
-            <!-- 左臂接口 -->
-            <xacro:cr5_interfaces name="left"/>
-            <!-- 右臂接口 -->
-            <xacro:cr5_interfaces name="right"/>
-            <!-- 夹爪接口 - 参考CR5的模块化设计 -->
-            <xacro:if value="${'$(arg type)' == 'AG2F90-C' or '$(arg type)' == 'AG2F90-C-Soft'}">
-                <xacro:include filename="$(find changingtek_description)/xacro/ros2_control/AG2F90-C.xacro"/>
-                <xacro:ag2f90c_interfaces name="left"/>
-                <xacro:ag2f90c_interfaces name="right"/>
-            </xacro:if>
-            <xacro:if value="${'$(arg type)' == 'robotiq85'}">
-                <xacro:include filename="$(find robotiq_description)/xacro/ros2_control/2F85.xacro"/>
-                <xacro:robotiq_2f85_interfaces name="left"/>
-                <xacro:robotiq_2f85_interfaces name="right"/>
-            </xacro:if>
-        </ros2_control>
-        <xacro:arg name="gazebo" default="false"/>
-        <xacro:if value="$(arg gazebo)">
-            <gazebo>
-                <plugin filename="gz_ros2_control-system" name="gz_ros2_control::GazeboSimROS2ControlPlugin">
-                    <parameters>$(find cr5_dual_description)/config/ros2_control/ros2_controllers.yaml</parameters>
-                </plugin>
-            </gazebo>
-            <!-- Gazebo configuration for CR5 dual arm -->
-        </xacro:if>
-    </xacro:if>
-    <xacro:if value="${'$(arg ros2_control_hardware_type)' == 'mock_components'}">
-        <!-- Mock Components: Unified ros2_control system -->
-        <ros2_control name="cr5_dual_system" type="system">
-            <hardware>
-                <plugin>mock_components/GenericSystem</plugin>
-            </hardware>
-            <!-- 左臂接口 -->
-            <xacro:cr5_interfaces name="left"/>
-            <!-- 右臂接口 -->
-            <xacro:cr5_interfaces name="right"/>
-            <!-- 夹爪接口 - 参考CR5的模块化设计 -->
-            <xacro:if value="${'$(arg type)' == 'AG2F90-C' or '$(arg type)' == 'AG2F90-C-Soft'}">
-                <xacro:include filename="$(find changingtek_description)/xacro/ros2_control/AG2F90-C.xacro"/>
-                <xacro:ag2f90c_interfaces name="left"/>
-                <xacro:ag2f90c_interfaces name="right"/>
-            </xacro:if>
-            <xacro:if value="${'$(arg type)' == 'robotiq85'}">
-                <xacro:include filename="$(find robotiq_description)/xacro/ros2_control/2F85.xacro"/>
-                <xacro:robotiq_2f85_interfaces name="left"/>
-                <xacro:robotiq_2f85_interfaces name="right"/>
-            </xacro:if>
-        </ros2_control>
-    </xacro:if>
+	<link name="world"/>
+	<joint name="world_fixed" type="fixed">
+		<parent link="world"/>
+		<child link="base_link"/>
+		<origin/>
+	</joint>
+	<!-- Include the base robot structure -->
+	<xacro:include filename="$(find cr5_dual_description)/xacro/robot.xacro"/>
+	<xacro:include filename="$(find cr5_description)/xacro/ros2_control/interfaces.xacro"/>
+	<xacro:if value="${'$(arg ros2_control_hardware_type)' == 'real'}">
+		<ros2_control name="cr5_left_system" type="system">
+			<hardware>
+				<plugin>dobot_ros2_control/DobotHardware</plugin>
+				<param name="robot_ip">192.168.5.33</param>
+				<param name="gain">200</param>
+				<param name="aheadtime">20</param>
+				<param name="speed_factor">100</param>
+				<param name="servo_time">0.3</param>
+			</hardware>
+			<xacro:cr5_interfaces name="left"/>
+			<xacro:if value="${'$(arg type)' != 'empty'}">
+				<joint name="left_gripper_joint">
+					<command_interface name="position"/>
+					<state_interface name="position">
+						<param name="initial_value">0</param>
+					</state_interface>
+				</joint>
+			</xacro:if>
+		</ros2_control>
+		<ros2_control name="cr5_right_system" type="system">
+			<hardware>
+				<plugin>dobot_ros2_control/DobotHardware</plugin>
+				<param name="robot_ip">192.168.5.34</param>
+				<param name="gain">200</param>
+				<param name="aheadtime">20</param>
+				<param name="speed_factor">100</param>
+				<param name="servo_time">0.3</param>
+			</hardware>
+			<xacro:cr5_interfaces name="right"/>
+			<xacro:if value="${'$(arg type)' != 'empty'}">
+				<joint name="right_gripper_joint">
+					<command_interface name="position"/>
+					<state_interface name="position">
+						<param name="initial_value">0</param>
+					</state_interface>
+				</joint>
+			</xacro:if>
+		</ros2_control>
+	</xacro:if>
+	<xacro:if value="${'$(arg ros2_control_hardware_type)' == 'isaac'}">
+		<!-- Isaac Sim: Use two separate topic_based systems for left and right arms -->
+		<ros2_control name="cr5_dual_system" type="system">
+			<hardware>
+				<plugin>topic_based_ros2_control/TopicBasedSystem</plugin>
+				<param name="joint_commands_topic">/isaac/joint_command</param>
+				<param name="joint_states_topic">/isaac/joint_states</param>
+				<param name="sum_wrapped_joint_states">false</param>
+				<param name="initialize_commands_from_state">true</param>
+			</hardware>
+			<!-- 左臂接口 -->
+			<xacro:cr5_interfaces name="left"/>
+			<!-- 右臂接口 -->
+			<xacro:cr5_interfaces name="right"/>
+			<!-- 夹爪接口 - 参考CR5的模块化设计 -->
+			<xacro:if value="${'$(arg type)' == 'AG2F90-C' or '$(arg type)' == 'AG2F90-C-Soft'}">
+				<xacro:include filename="$(find changingtek_description)/xacro/ros2_control/AG2F90-C.xacro"/>
+				<xacro:ag2f90c_interfaces name="left"/>
+				<xacro:ag2f90c_interfaces name="right"/>
+			</xacro:if>
+			<xacro:if value="${'$(arg type)' == 'robotiq85'}">
+				<xacro:include filename="$(find robotiq_description)/xacro/ros2_control/2F85.xacro"/>
+				<xacro:robotiq_2f85_interfaces name="left"/>
+				<xacro:robotiq_2f85_interfaces name="right"/>
+			</xacro:if>
+		</ros2_control>
+	</xacro:if>
+	<xacro:if value="${'$(arg ros2_control_hardware_type)' == 'gz'}">
+		<!-- Gazebo Simulator: Unified ros2_control system -->
+		<ros2_control name="cr5_dual_system" type="system">
+			<hardware>
+				<plugin>gz_ros2_control/GazeboSimSystem</plugin>
+			</hardware>
+			<!-- 左臂接口 -->
+			<xacro:cr5_interfaces name="left"/>
+			<!-- 右臂接口 -->
+			<xacro:cr5_interfaces name="right"/>
+			<!-- 夹爪接口 - 参考CR5的模块化设计 -->
+			<xacro:if value="${'$(arg type)' == 'AG2F90-C' or '$(arg type)' == 'AG2F90-C-Soft'}">
+				<xacro:include filename="$(find changingtek_description)/xacro/ros2_control/AG2F90-C.xacro"/>
+				<xacro:ag2f90c_interfaces name="left"/>
+				<xacro:ag2f90c_interfaces name="right"/>
+			</xacro:if>
+			<xacro:if value="${'$(arg type)' == 'robotiq85'}">
+				<xacro:include filename="$(find robotiq_description)/xacro/ros2_control/2F85.xacro"/>
+				<xacro:robotiq_2f85_interfaces name="left"/>
+				<xacro:robotiq_2f85_interfaces name="right"/>
+			</xacro:if>
+		</ros2_control>
+		<xacro:arg name="gazebo" default="false"/>
+		<xacro:if value="$(arg gazebo)">
+			<gazebo>
+				<plugin filename="gz_ros2_control-system" name="gz_ros2_control::GazeboSimROS2ControlPlugin">
+					<parameters>$(find cr5_dual_description)/config/ros2_control/ros2_controllers.yaml</parameters>
+				</plugin>
+			</gazebo>
+			<!-- Gazebo configuration for CR5 dual arm -->
+		</xacro:if>
+	</xacro:if>
+	<xacro:if value="${'$(arg ros2_control_hardware_type)' == 'mock_components'}">
+		<!-- Mock Components: Unified ros2_control system -->
+		<ros2_control name="cr5_dual_system" type="system">
+			<hardware>
+				<plugin>mock_components/GenericSystem</plugin>
+			</hardware>
+			<!-- 左臂接口 -->
+			<xacro:cr5_interfaces name="left"/>
+			<!-- 右臂接口 -->
+			<xacro:cr5_interfaces name="right"/>
+			<!-- 夹爪接口 - 参考CR5的模块化设计 -->
+			<xacro:if value="${'$(arg type)' == 'AG2F90-C' or '$(arg type)' == 'AG2F90-C-Soft'}">
+				<xacro:include filename="$(find changingtek_description)/xacro/ros2_control/AG2F90-C.xacro"/>
+				<xacro:ag2f90c_interfaces name="left"/>
+				<xacro:ag2f90c_interfaces name="right"/>
+			</xacro:if>
+			<xacro:if value="${'$(arg type)' == 'robotiq85'}">
+				<xacro:include filename="$(find robotiq_description)/xacro/ros2_control/2F85.xacro"/>
+				<xacro:robotiq_2f85_interfaces name="left"/>
+				<xacro:robotiq_2f85_interfaces name="right"/>
+			</xacro:if>
+		</ros2_control>
+	</xacro:if>
 </robot>
