Commit message: add vla 39 config

File: cr5_description/xacro/grippers.xacro (robot description, xacro)
@@ -1,7 +1,11 @@
 <?xml version="1.0"?>
 <robot name="DobotCR5" xmlns:xacro="http://www.ros.org/wiki/xacro">
-	<xacro:arg name="type" default="empty"/>
+	<!--
+	  夹爪类型由 cr5_description/xacro/robot.xacro 解析得到：
+	  - selected_gripper_type: empty / robotiq85 / AG2F90-C(-Soft) / AG2F120S ...
+	  - selected_scene: 可选（当前文件不使用）
+	-->
 	<!-- 根据type参数决定使用哪种夹爪 -->
-	<xacro:if value="${'$(arg type)' == 'robotiq85'}">
+	<xacro:if value="${selected_gripper_type == 'robotiq85'}">
 		<xacro:include filename="$(find robotiq_description)/xacro/2F85.xacro"/>
 		<xacro:Robotiq85 name=""/>
@@ -11,5 +15,5 @@
 		</joint>
 	</xacro:if>
-	<xacro:if value="${'$(arg type)' == 'AG2F90-C'}">
+	<xacro:if value="${selected_gripper_type == 'AG2F90-C'}">
 		<xacro:include filename="$(find changingtek_description)/xacro/AG2F90-C.xacro"/>
 		<xacro:AG2F90-C name="" use_flange="true"/>
@@ -20,5 +24,5 @@
 		</joint>
 	</xacro:if>
-	<xacro:if value="${'$(arg type)' == 'AG2F90-C-Soft'}">
+	<xacro:if value="${selected_gripper_type == 'AG2F90-C-Soft'}">
 		<xacro:include filename="$(find changingtek_description)/xacro/AG2F90-C.xacro"/>
 		<xacro:AG2F90-C name="" use_flange="true" pad="soft"/>
@@ -35,5 +39,5 @@
 		</joint>
 	</xacro:if>
-	<xacro:if value="${'$(arg type)' == 'AG2F120S'}">
+	<xacro:if value="${selected_gripper_type == 'AG2F120S'}">
 		<xacro:include filename="$(find changingtek_description)/xacro/AG2F120S.xacro"/>
 		<xacro:AG2F120S name=""/>

File: cr5_description/xacro/robot.xacro (robot description, xacro)
@@ -2,4 +2,52 @@
 <robot name="DobotCR5" xmlns:xacro="http://www.ros.org/wiki/xacro">
   <xacro:arg name="collider" default="convex"/>
+  <xacro:arg name="type" default="empty"/>
+  <xacro:arg name="scene" default=""/>
+  <!--
+    CR5 的 type 不仅用于末端夹爪，也可承载场景(scene)信息（类似 m6_ccs_description 的机制）。
+    - 兼容：type=AG2F90-C-Soft / robotiq85 / empty 等老用法
+    - 扩展：type=usb-90c / desktop_90c 等会同时设置 selected_scene + selected_gripper_type
+  -->
+  <xacro:property name="type_arg" value="$(arg type)"/>
+  <!-- 默认值 -->
+  <xacro:property name="selected_gripper_type" value="empty"/>
+  <xacro:property name="selected_scene" value=""/>
+  <!-- 夹爪解析（保持与历史 type 值一致） -->
+  <xacro:if value="${type_arg == 'robotiq85'}">
+    <xacro:property name="selected_gripper_type" value="robotiq85"/>
+  </xacro:if>
+  <xacro:if value="${type_arg == 'AG2F90-C'}">
+    <xacro:property name="selected_gripper_type" value="AG2F90-C"/>
+  </xacro:if>
+  <xacro:if value="${type_arg == 'AG2F90-C-Soft'}">
+    <xacro:property name="selected_gripper_type" value="AG2F90-C-Soft"/>
+  </xacro:if>
+  <xacro:if value="${type_arg == 'AG2F120S'}">
+    <xacro:property name="selected_gripper_type" value="AG2F120S"/>
+  </xacro:if>
+  <xacro:if value="${type_arg == 'empty' or type_arg == ''}">
+    <xacro:property name="selected_gripper_type" value="empty"/>
+  </xacro:if>
+  <!-- 场景 + 夹爪的复合 type（可按需继续扩展） -->
+  <xacro:if value="${type_arg == 'vla39'}">
+    <xacro:property name="selected_scene" value="vla39"/>
+    <xacro:property name="selected_gripper_type" value="AG2F90-C-Soft"/>
+  </xacro:if>
+  <xacro:if value="${type_arg == 'usb-90c'}">
+    <xacro:property name="selected_scene" value="usb-90c"/>
+    <!-- Dobot 默认使用 90C（软爪） -->
+    <xacro:property name="selected_gripper_type" value="AG2F90-C-Soft"/>
+  </xacro:if>
+  <xacro:if value="${type_arg == 'desktop'}">
+    <xacro:property name="selected_scene" value="desktop"/>
+  </xacro:if>
+  <xacro:if value="${type_arg == 'desktop_90c'}">
+    <xacro:property name="selected_scene" value="desktop"/>
+    <xacro:property name="selected_gripper_type" value="AG2F90-C-Soft"/>
+  </xacro:if>
+  <!-- 允许显式传入 scene 覆盖（如果你愿意用 scene:=xxx） -->
+  <xacro:if value="${'$(arg scene)' != ''}">
+    <xacro:property name="selected_scene" value="$(arg scene)"/>
+  </xacro:if>
   <!-- 从同目录下的tf_params.yaml文件加载tf参数 -->
   <xacro:property name="tf_params" value="${xacro.load_yaml('$(find cr5_description)/xacro/tf_params.yaml')['tf_params']}"/>

File: cr5_description/xacro/ros2_control/interfaces.xacro (robot description, xacro)
@@ -7,5 +7,5 @@
         <command_interface name="position"/>
         <state_interface name="position">
-          <param name="initial_value">0</param>
+          <param name="initial_value">3.14159</param>
         </state_interface>
         <state_interface name="velocity"/>

File: cr5_description/xacro/ros2_control/robot.xacro (robot description, xacro)
@@ -27,9 +27,14 @@
       <xacro:if value="${'$(arg ros2_control_hardware_type)' == 'real'}">
         <plugin>dobot_ros2_control/DobotHardware</plugin>
-        <param name="robot_ip">192.168.5.34</param>
+        <xacro:if value="${selected_scene == 'vla39'}">
+          <param name="robot_ip">192.168.5.39</param>
+        </xacro:if>
+        <xacro:if value="${selected_scene == ''}">
+          <param name="robot_ip">192.168.5.34</param>
+        </xacro:if>
         <param name="gain">800</param>
         <param name="aheadtime">50</param>
         <param name="speed_factor">100</param>
-        <param name="servo_time">0.5</param>
+        <param name="servo_time">0.05</param>
       </xacro:if>
     </hardware>
@@ -38,5 +43,5 @@
     <xacro:if value="${'$(arg ros2_control_hardware_type)' == 'real'}">
       <!-- 真实硬件模式：使用简单的gripper joint，仅有位置接口 -->
-      <xacro:if value="${'$(arg type)' == 'AG2F90-C-Soft'}">
+      <xacro:if value="${selected_gripper_type == 'AG2F90-C-Soft'}">
         <joint name="gripper_joint">
           <command_interface name="position"/>
@@ -49,13 +54,13 @@
     <xacro:unless value="${'$(arg ros2_control_hardware_type)' == 'real'}">
       <!-- 非真实硬件模式：使用现有的夹爪定义 -->
-      <xacro:if value="${'$(arg type)' == 'AG2F90-C' or '$(arg type)' == 'AG2F90-C-Soft'}">
+      <xacro:if value="${selected_gripper_type == 'AG2F90-C' or selected_gripper_type == 'AG2F90-C-Soft'}">
         <xacro:include filename="$(find changingtek_description)/xacro/ros2_control/AG2F90-C.xacro"/>
         <xacro:ag2f90c_interfaces name=""/>
       </xacro:if>
-      <xacro:if value="${'$(arg type)' == 'AG2F120S'}">
+      <xacro:if value="${selected_gripper_type == 'AG2F120S'}">
         <xacro:include filename="$(find changingtek_description)/xacro/ros2_control/AG2F120S.xacro"/>
         <xacro:ag2f120s_interfaces name=""/>
       </xacro:if>
-      <xacro:if value="${'$(arg type)' == 'robotiq85'}">
+      <xacro:if value="${selected_gripper_type == 'robotiq85'}">
         <xacro:include filename="$(find robotiq_description)/xacro/ros2_control/2F85.xacro"/>
         <xacro:robotiq_2f85_interfaces name=""/>

File: cr5_dual_description/xacro/grippers.xacro (robot description, xacro)
@@ -1,7 +1,7 @@
 <?xml version="1.0"?>
 <robot name="DobotCR5" xmlns:xacro="http://www.ros.org/wiki/xacro">
-  <xacro:arg name="type" default="empty"/>
+  <!-- 夹爪类型由 cr5_dual_description/xacro/robot.xacro 解析得到：selected_gripper_type -->
   <!-- 根据type参数决定使用哪种夹爪 -->
-  <xacro:if value="${'$(arg type)' == 'robotiq85'}">
+  <xacro:if value="${selected_gripper_type == 'robotiq85'}">
     <xacro:include filename="$(find robotiq_description)/xacro/2F85.xacro"/>
     <xacro:Robotiq85 name="left"/>
@@ -16,5 +16,5 @@
     </joint>
   </xacro:if>
-  <xacro:if value="${'$(arg type)' == 'AG2F90-C-Soft'}">
+  <xacro:if value="${selected_gripper_type == 'AG2F90-C-Soft'}">
     <xacro:include filename="$(find changingtek_description)/xacro/AG2F90-C.xacro"/>
     <xacro:AG2F90-C name="left" use_flange="true" pad="soft"/>
@@ -31,5 +31,5 @@
     </joint>
   </xacro:if>
-  <xacro:if value="${'$(arg type)' == 'AG2F90-C'}">
+  <xacro:if value="${selected_gripper_type == 'AG2F90-C'}">
     <xacro:include filename="$(find changingtek_description)/xacro/AG2F90-C.xacro"/>
     <xacro:AG2F90-C name="left" use_flange="true"/>

File: cr5_dual_description/xacro/robot.xacro (robot description, xacro)
@@ -2,4 +2,32 @@
 <robot name="DobotCR5_Dual" xmlns:xacro="http://www.ros.org/wiki/xacro">
   <xacro:arg name="collider" default="convex"/>
+  <xacro:arg name="type" default="empty"/>
+  <xacro:arg name="scene" default=""/>
+  <!-- 与单臂一致：解析 type 得到 selected_gripper_type + selected_scene -->
+  <xacro:property name="type_arg" value="$(arg type)"/>
+  <xacro:property name="selected_gripper_type" value="empty"/>
+  <xacro:property name="selected_scene" value=""/>
+  <xacro:if value="${type_arg == 'robotiq85'}">
+    <xacro:property name="selected_gripper_type" value="robotiq85"/>
+  </xacro:if>
+  <xacro:if value="${type_arg == 'AG2F90-C'}">
+    <xacro:property name="selected_gripper_type" value="AG2F90-C"/>
+  </xacro:if>
+  <xacro:if value="${type_arg == 'AG2F90-C-Soft'}">
+    <xacro:property name="selected_gripper_type" value="AG2F90-C-Soft"/>
+  </xacro:if>
+  <xacro:if value="${type_arg == 'empty' or type_arg == ''}">
+    <xacro:property name="selected_gripper_type" value="empty"/>
+  </xacro:if>
+  <xacro:if value="${type_arg == 'dual_desktop'}">
+    <xacro:property name="selected_scene" value="desktop"/>
+  </xacro:if>
+  <xacro:if value="${type_arg == 'dual_desktop_90c'}">
+    <xacro:property name="selected_scene" value="desktop"/>
+    <xacro:property name="selected_gripper_type" value="AG2F90-C-Soft"/>
+  </xacro:if>
+  <xacro:if value="${'$(arg scene)' != ''}">
+    <xacro:property name="selected_scene" value="$(arg scene)"/>
+  </xacro:if>
   <xacro:property name="tf_params" value="${xacro.load_yaml('$(find cr5_description)/xacro/tf_params.yaml')['tf_params']}"/>
   <link name="base_link">

File: cr5_dual_description/xacro/ros2_control/robot.xacro (robot description, xacro)
@@ -21,5 +21,5 @@
 			</hardware>
 			<xacro:cr5_interfaces name="left"/>
-			<xacro:if value="${'$(arg type)' != 'empty'}">
+			<xacro:if value="${selected_gripper_type != 'empty'}">
 				<joint name="left_gripper_joint">
 					<command_interface name="position"/>
@@ -40,5 +40,5 @@
 			</hardware>
 			<xacro:cr5_interfaces name="right"/>
-			<xacro:if value="${'$(arg type)' != 'empty'}">
+			<xacro:if value="${selected_gripper_type != 'empty'}">
 				<joint name="right_gripper_joint">
 					<command_interface name="position"/>
@@ -65,10 +65,10 @@
 			<xacro:cr5_interfaces name="right"/>
 			<!-- 夹爪接口 - 参考CR5的模块化设计 -->
-			<xacro:if value="${'$(arg type)' == 'AG2F90-C' or '$(arg type)' == 'AG2F90-C-Soft'}">
+			<xacro:if value="${selected_gripper_type == 'AG2F90-C' or selected_gripper_type == 'AG2F90-C-Soft'}">
 				<xacro:include filename="$(find changingtek_description)/xacro/ros2_control/AG2F90-C.xacro"/>
 				<xacro:ag2f90c_interfaces name="left"/>
 				<xacro:ag2f90c_interfaces name="right"/>
 			</xacro:if>
-			<xacro:if value="${'$(arg type)' == 'robotiq85'}">
+			<xacro:if value="${selected_gripper_type == 'robotiq85'}">
 				<xacro:include filename="$(find robotiq_description)/xacro/ros2_control/2F85.xacro"/>
 				<xacro:robotiq_2f85_interfaces name="left"/>
@@ -88,10 +88,10 @@
 			<xacro:cr5_interfaces name="right"/>
 			<!-- 夹爪接口 - 参考CR5的模块化设计 -->
-			<xacro:if value="${'$(arg type)' == 'AG2F90-C' or '$(arg type)' == 'AG2F90-C-Soft'}">
+			<xacro:if value="${selected_gripper_type == 'AG2F90-C' or selected_gripper_type == 'AG2F90-C-Soft'}">
 				<xacro:include filename="$(find changingtek_description)/xacro/ros2_control/AG2F90-C.xacro"/>
 				<xacro:ag2f90c_interfaces name="left"/>
 				<xacro:ag2f90c_interfaces name="right"/>
 			</xacro:if>
-			<xacro:if value="${'$(arg type)' == 'robotiq85'}">
+			<xacro:if value="${selected_gripper_type == 'robotiq85'}">
 				<xacro:include filename="$(find robotiq_description)/xacro/ros2_control/2F85.xacro"/>
 				<xacro:robotiq_2f85_interfaces name="left"/>
@@ -120,10 +120,10 @@
 			<xacro:cr5_interfaces name="right"/>
 			<!-- 夹爪接口 - 参考CR5的模块化设计 -->
-			<xacro:if value="${'$(arg type)' == 'AG2F90-C' or '$(arg type)' == 'AG2F90-C-Soft'}">
+			<xacro:if value="${selected_gripper_type == 'AG2F90-C' or selected_gripper_type == 'AG2F90-C-Soft'}">
 				<xacro:include filename="$(find changingtek_description)/xacro/ros2_control/AG2F90-C.xacro"/>
 				<xacro:ag2f90c_interfaces name="left"/>
 				<xacro:ag2f90c_interfaces name="right"/>
 			</xacro:if>
-			<xacro:if value="${'$(arg type)' == 'robotiq85'}">
+			<xacro:if value="${selected_gripper_type == 'robotiq85'}">
 				<xacro:include filename="$(find robotiq_description)/xacro/ros2_control/2F85.xacro"/>
 				<xacro:robotiq_2f85_interfaces name="left"/>

Commit message: ocs2_admittance config update

File: cr5_description/xacro/grippers.xacro (robot description, xacro)
@@ -14,8 +14,20 @@
 		<xacro:include filename="$(find changingtek_description)/xacro/AG2F90-C.xacro"/>
 		<xacro:AG2F90-C name="" use_flange="true"/>
+		<link name="ft_sensor">
+			<visual>
+				<geometry>
+					<mesh filename="file://$(find cr5_description)/meshes/visual/ft_sensor.obj"/>
+				</geometry>
+			</visual>
+		</link>
+		<joint name="ft_sensor_joint" type="fixed">
+			<origin rpy="0 0 ${PI}"/>
+			<parent link="Link6"/>
+			<child link="ft_sensor"/>
+		</joint>
 		<joint name="gripper_fix" type="fixed">
-			<parent link="Link6"/>
+			<parent link="ft_sensor"/>
 			<child link="flange"/>
-			<origin rpy="0 0 ${-PI/2}"/>
+			<origin xyz="0 0 0.037" rpy="0 0 ${-PI/2}"/>
 		</joint>
 	</xacro:if>
@@ -23,8 +35,20 @@
 		<xacro:include filename="$(find changingtek_description)/xacro/AG2F90-C.xacro"/>
 		<xacro:AG2F90-C name="" use_flange="true" pad="soft"/>
+		<link name="ft_sensor">
+			<visual>
+				<geometry>
+					<mesh filename="file://$(find cr5_description)/meshes/visual/ft_sensor.obj"/>
+				</geometry>
+			</visual>
+		</link>
+		<joint name="ft_sensor_joint" type="fixed">
+			<origin rpy="0 0 ${PI}"/>
+			<parent link="Link6"/>
+			<child link="ft_sensor"/>
+		</joint>
 		<joint name="gripper_fix" type="fixed">
-			<parent link="Link6"/>
+			<parent link="ft_sensor"/>
 			<child link="flange"/>
-			<origin rpy="0 0 ${PI/2}"/>
+			<origin xyz="0 0 0.037" rpy="0 0 ${PI/2}"/>
 		</joint>
 	</xacro:if>
@@ -47,5 +71,5 @@
 		</link>
 		<joint name="ft_sensor_joint" type="fixed">
-			<origin rpy="0 0 ${PI}"/>
+			<origin rpy="0 0 ${-PI/2}"/>
 			<parent link="Link6"/>
 			<child link="ft_sensor"/>

File: cr5_description/xacro/ros2_control/robot.xacro (robot description, xacro)
@@ -2,4 +2,8 @@
 <robot xmlns:xacro="http://www.ros.org/wiki/xacro" name="CR5">
     <xacro:arg name="ros2_control_hardware_type" default="mock_components"/>
+    <xacro:arg name="force_control_mode" default="ros2_control_controllers"/>
+    <xacro:arg name="enable_servoj_stream" default="true"/>
+    <xacro:arg name="allow_servoj_with_force_drag" default="false"/>
+    <xacro:arg name="enable_gripper_io" default="true"/>
     <link name="world"/>
     <joint name="world_fixed" type="fixed">
@@ -32,4 +36,10 @@
                 <param name="speed_factor">1</param>
                 <param name="servo_time">0.02</param>
+                <param name="force_control_mode">$(arg force_control_mode)</param>
+                <param name="force_service_prefix">dobot_force_control/srv</param>
+                <param name="enable_servoj_stream">$(arg enable_servoj_stream)</param>
+                <param name="allow_servoj_with_force_drag">$(arg allow_servoj_with_force_drag)</param>
+                <param name="enable_gripper_io">$(arg enable_gripper_io)</param>
+                <param name="gripper_read_frequency_divider">100</param>
             </xacro:if>
         </hardware>
@@ -38,5 +48,5 @@
         <xacro:if value="${'$(arg ros2_control_hardware_type)' == 'real'}">
             <!-- 真实硬件模式：使用简单的gripper joint，仅有位置接口 -->
-            <xacro:if value="${'$(arg type)' != 'empty'}">
+            <xacro:if value="${('$(arg type)' == 'ft-90c' or '$(arg type)' == 'AG2F90-C' or '$(arg type)' == 'AG2F90-C-Soft' or '$(arg type)' == 'robotiq85') and '$(arg enable_gripper_io)' == 'true'}">
                 <joint name="gripper_joint">
                     <command_interface name="position"/>
@@ -46,5 +56,5 @@
                 </joint>
             </xacro:if>
-            <xacro:if value="${'$(arg type)' == 'ft-90c'}">
+            <xacro:if value="${'$(arg type)' == 'ft-90c' or '$(arg type)' == 'AG2F90-C' or '$(arg type)' == 'AG2F90-C-Soft' or '$(arg type)' == 'robotiq85'}">
                 <!-- 六维力传感器定义 -->
                 <sensor name="ft_sensor">

File: cr5_dual_description/xacro/ros2_control/robot.xacro (robot description, xacro)
@@ -1,4 +1,7 @@
 <?xml version="1.0" ?>
 <robot name="fiveages_cr5_dual_station" xmlns:xacro="http://www.ros.org/wiki/xacro">
+    <xacro:arg name="force_control_mode" default="ros2_control_controllers"/>
+    <xacro:arg name="enable_servoj_stream" default="true"/>
+    <xacro:arg name="enable_gripper_io" default="true"/>
     <link name="world"/>
     <joint name="world_fixed" type="fixed">
@@ -20,4 +23,8 @@
                 <param name="servo_time">0.05</param>
                 <param name="gripper_read_frequency_divider">50</param>
+                <param name="force_control_mode">$(arg force_control_mode)</param>
+                <param name="force_service_prefix">left_dobot_force_control/srv</param>
+                <param name="enable_servoj_stream">$(arg enable_servoj_stream)</param>
+                <param name="enable_gripper_io">$(arg enable_gripper_io)</param>
             </hardware>
             <xacro:cr5_interfaces name="left"/>
@@ -48,4 +55,8 @@
                     <param name="speed_factor">100</param>
                     <param name="servo_time">0.3</param>
+                    <param name="force_control_mode">$(arg force_control_mode)</param>
+                    <param name="force_service_prefix">right_dobot_force_control/srv</param>
+                    <param name="enable_servoj_stream">$(arg enable_servoj_stream)</param>
+                    <param name="enable_gripper_io">$(arg enable_gripper_io)</param>
                 </hardware>
                 <xacro:cr5_interfaces name="right"/>
