Commit message: ft 90c and cartesian controller

File: cr5_description/xacro/arm.xacro (robot description, xacro)
@@ -1,294 +1,301 @@
 <?xml version="1.0"?>
 <robot name="cr5_robot" xmlns:xacro="http://ros.org/wiki/xacro">
-	<xacro:property name="PI" value="3.1415926535897931"/>
-	<xacro:macro name="CR5" params="name collider:=convex">
-		<xacro:property name="prefix" value="${name + '_' if name else ''}"/>
-		<link name="${prefix}base_link">
-			<inertial>
-				<origin xyz="-8.0961E-06 0.0019103 0.028995"/>
-				<mass value="0.90882"/>
-			<inertia ixx="0.0014545" ixy="4.2968E-08" ixz="-1.8199E-07" iyy="0.001345" iyz="-6.243E-06" izz="0.002155"/>
-			</inertial>
-			<visual>
-				<geometry>
-					<mesh filename="file://$(find cr5_description)/meshes/visual/base_link.obj"/>
-				</geometry>
-			</visual>
-			<xacro:if value="${collider == 'convex'}">
-				<collision>
-					<geometry>
-						<mesh filename="file://$(find cr5_description)/meshes/collision/base_link.stl"/>
-					</geometry>
-				</collision>
-			</xacro:if>
-			<xacro:if value="${collider == 'simple'}">
-				<collision>
-					<origin xyz="0 0 0.05"/>
-					<geometry>
-						<cylinder length="0.1" radius="0.1"/>
-					</geometry>
-				</collision>
-				<xacro:if value="${prefix == ''}">
-					<collision>
-						<origin xyz="0 0 -0.025"/>
-						<geometry>
-							<box size="1.5 1.5 0.05"/>
-						</geometry>
-					</collision>
-				</xacro:if>
-			</xacro:if>
-		</link>
-		<link name="${prefix}Link1">
-			<inertial>
-				<origin xyz="-8.7268E-07 -0.0032576 -0.0076748"/>
-				<mass value="1.6123"/>
-			<inertia ixx="0.0029122" ixy="5.7387E-09" ixz="1.9945E-08" iyy="0.0028191" iyz="0.00044094" izz="0.0032836"/>
-			</inertial>
-			<visual>
-				<geometry>
-					<mesh filename="file://$(find cr5_description)/meshes/visual/Link1.obj"/>
-				</geometry>
-			</visual>
-			<xacro:if value="${collider == 'convex'}">
-				<collision>
-					<geometry>
-						<mesh filename="file://$(find cr5_description)/meshes/collision/Link1_0.stl"/>
-					</geometry>
-				</collision>
-				<collision>
-					<geometry>
-						<mesh filename="file://$(find cr5_description)/meshes/collision/Link1_1.stl"/>
-					</geometry>
-				</collision>
-			</xacro:if>
-			<xacro:if value="${collider == 'simple'}">
-				<collision>
-					<geometry>
-						<cylinder length="0.17" radius="0.08"/>
-					</geometry>
-				</collision>
-			</xacro:if>
-		</link>
-	<joint name="${prefix}joint1" type="revolute">
-		<origin xyz="0 0 0.147"/>
-		<parent link="${prefix}base_link"/>
-		<child link="${prefix}Link1"/>
-			<axis xyz="0 0 1"/>
-			<limit lower="${-2*PI}" upper="${2*PI}" effort="300" velocity="${PI}"/>
-		</joint>
-		<link name="${prefix}Link2">
-			<inertial>
-				<origin xyz="-0.21351 -1.3842E-06 0.14252"/>
-				<mass value="5.5186"/>
-			<inertia ixx="0.0085919" ixy="7.5552E-07" ixz="-7.8922E-07" iyy="0.027553" iyz="1.4629E-07" izz="0.028294"/>
-			</inertial>
-			<visual>
-				<geometry>
-					<mesh filename="file://$(find cr5_description)/meshes/visual/Link2.obj"/>
-				</geometry>
-			</visual>
-			<xacro:if value="${collider == 'convex'}">
-				<collision>
-					<geometry>
-						<mesh filename="file://$(find cr5_description)/meshes/collision/Link2_0.stl"/>
-					</geometry>
-				</collision>
-				<collision>
-					<geometry>
-						<mesh filename="file://$(find cr5_description)/meshes/collision/Link2_1.stl"/>
-					</geometry>
-				</collision>
-				<collision>
-					<geometry>
-						<mesh filename="file://$(find cr5_description)/meshes/collision/Link2_2.stl"/>
-					</geometry>
-				</collision>
-			</xacro:if>
-			<xacro:if value="${collider == 'simple'}">
-				<collision>
-					<origin rpy="0 0 0" xyz="0 0 0.145"/>
-					<geometry>
-						<cylinder length="0.18" radius="0.07"/>
-					</geometry>
-				</collision>
-				<collision>
-					<origin rpy="0 ${PI/2} 0" xyz="-0.2 0 0.15"/>
-					<geometry>
-						<cylinder length="0.43" radius="0.065"/>
-					</geometry>
-				</collision>
-				<collision>
-					<origin xyz="-0.43 0 0.145"/>
-					<geometry>
-						<cylinder length="0.18" radius="0.07"/>
-					</geometry>
-				</collision>
-			</xacro:if>
-		</link>
-	<joint name="${prefix}joint2" type="revolute">
-		<origin rpy="${PI/2} ${PI/2} 0"/>
-		<parent link="${prefix}Link1"/>
-		<child link="${prefix}Link2"/>
-			<axis xyz="0 0 1"/>
-			<limit lower="${-2*PI}" upper="${2*PI}" effort="300" velocity="${PI}"/>
-		</joint>
-		<link name="${prefix}Link3">
-			<inertial>
-				<origin xyz="-0.15231 -1.4079E-07 0.022693"/>
-				<mass value="2.8536"/>
-			<inertia ixx="0.0032608" ixy="-3.2147E-10" ixz="0.00012363" iyy="0.0092967" iyz="2.9478E-10" izz="0.0095552"/>
-			</inertial>
-			<visual>
-				<geometry>
-					<mesh filename="file://$(find cr5_description)/meshes/visual/Link3.obj"/>
-				</geometry>
-			</visual>
-			<xacro:if value="${collider == 'convex'}">
-				<collision>
-					<geometry>
-						<mesh filename="file://$(find cr5_description)/meshes/collision/Link3_0.stl"/>
-					</geometry>
-				</collision>
-				<collision>
-					<geometry>
-						<mesh filename="file://$(find cr5_description)/meshes/collision/Link3_1.stl"/>
-					</geometry>
-				</collision>
-				<collision>
-					<geometry>
-						<mesh filename="file://$(find cr5_description)/meshes/collision/Link3_2.stl"/>
-					</geometry>
-				</collision>
-			</xacro:if>
-			<xacro:if value="${collider == 'simple'}">
-				<collision>
-					<origin xyz="0 0 0.02"/>
-					<geometry>
-						<cylinder length="0.15" radius="0.07"/>
-					</geometry>
-				</collision>
-				<collision>
-					<origin rpy="0 ${PI/2} 0" xyz="-0.2 0 0.03"/>
-					<geometry>
-						<cylinder length="0.26" radius="0.05"/>
-					</geometry>
-				</collision>
-				<collision>
-					<origin xyz="-0.355 0 0.02"/>
-					<geometry>
-						<cylinder length="0.15" radius="0.05"/>
-					</geometry>
-				</collision>
-			</xacro:if>
-		</link>
-	<joint name="${prefix}joint3" type="revolute">
-		<origin xyz="-0.427 0 0"/>
-		<parent link="${prefix}Link2"/>
-		<child link="${prefix}Link3"/>
-			<axis xyz="0 0 1"/>
-			<limit lower="-2.7925" upper="2.7925" effort="300" velocity="3.14159"/>
-		</joint>
-		<link name="${prefix}Link4">
-			<inertial>
-				<origin xyz="-3.2386E-07 -0.002077 -0.0015548"/>
-				<mass value="0.67058"/>
-			<inertia ixx="0.00066939" ixy="4.1975E-10" ixz="-1.0734E-08" iyy="0.00065424" iyz="0.00011081" izz="0.00065365"/>
-			</inertial>
-			<visual>
-				<geometry>
-					<mesh filename="file://$(find cr5_description)/meshes/visual/Link4.obj"/>
-				</geometry>
-			</visual>
-			<xacro:if value="${collider == 'convex'}">
-				<collision>
-					<geometry>
-						<mesh filename="file://$(find cr5_description)/meshes/collision/Link4.stl"/>
-					</geometry>
-				</collision>
-			</xacro:if>
-			<xacro:if value="${collider == 'simple'}">
-				<collision>
-					<origin rpy="${PI/2} 0 0"/>
-					<geometry>
-						<cylinder length="0.155" radius="0.055"/>
-					</geometry>
-				</collision>
-			</xacro:if>
-		</link>
-	<joint name="${prefix}joint4" type="revolute">
-		<origin xyz="-0.357 0 0.141" rpy="0 0 ${-PI/2}"/>
-		<parent link="${prefix}Link3"/>
-		<child link="${prefix}Link4"/>
-			<axis xyz="0 0 1"/>
-			<limit lower="${-2*PI}" upper="${2*PI}" effort="300" velocity="${PI}"/>
-		</joint>
-		<link name="${prefix}Link5">
-			<inertial>
-				<origin xyz="-3.7738E-07 -0.0045777 -0.0012971"/>
-				<mass value="0.7269"/>
-			<inertia ixx="0.00073069" ixy="-5.7806E-09" ixz="6.7132E-09" iyy="0.00071195" iyz="-0.00011926" izz="0.00071391"/>
-			</inertial>
-			<visual>
-				<geometry>
-					<mesh filename="file://$(find cr5_description)/meshes/visual/Link5.obj"/>
-				</geometry>
-			</visual>
-			<xacro:if value="${collider == 'convex'}">
-				<collision>
-					<geometry>
-						<mesh filename="file://$(find cr5_description)/meshes/collision/Link5.stl"/>
-					</geometry>
-				</collision>
-			</xacro:if>
-			<xacro:if value="${collider == 'simple'}">
-				<collision>
-					<origin rpy="${PI/2} 0 0"/>
-					<geometry>
-						<cylinder length="0.18" radius="0.055"/>
-					</geometry>
-				</collision>
-			</xacro:if>
-		</link>
-	<joint name="${prefix}joint5" type="revolute">
-		<origin xyz="0 -0.116 0" rpy="${PI/2} 0 0"/>
-		<parent link="${prefix}Link4"/>
-		<child link="${prefix}Link5"/>
-			<axis xyz="0 0 1"/>
-			<limit lower="${-2*PI}" upper="${2*PI}" effort="300" velocity="${PI}"/>
-		</joint>
-		<link name="${prefix}Link6">
-			<inertial>
-				<origin xyz="5.0777E-11 9.3774E-05 -0.019285"/>
-				<mass value="0.15789"/>
-			<inertia ixx="7.8045E-05" ixy="6.1582E-15" ixz="6.2471E-14" iyy="7.9168E-05" iyz="-1.3822E-07" izz="0.00012951"/>
-			</inertial>
-			<visual>
-				<geometry>
-					<mesh filename="file://$(find cr5_description)/meshes/visual/Link6.obj"/>
-				</geometry>
-			</visual>
-			<xacro:if value="${collider == 'convex'}">
-				<collision>
-					<geometry>
-						<mesh filename="file://$(find cr5_description)/meshes/collision/Link6.stl"/>
-					</geometry>
-				</collision>
-			</xacro:if>
-			<xacro:if value="${collider == 'simple'}">
-				<collision>
-					<origin xyz="0 0 0.1"/>
-					<geometry>
-						<box size="0.05 0.15 0.2"/>
-					</geometry>
-				</collision>
-			</xacro:if>
-		</link>
-	<joint name="${prefix}joint6" type="revolute">
-		<origin xyz="0 0.105 0" rpy="${-PI/2} 0 0"/>
-		<parent link="${prefix}Link5"/>
-		<child link="${prefix}Link6"/>
-			<axis xyz="0 0 1"/>
-			<limit lower="${-2*PI}" upper="${2*PI}" effort="300" velocity="${PI}"/>
-		</joint>
-	</xacro:macro>
+    <xacro:property name="PI" value="3.1415926535897931"/>
+    <xacro:macro name="CR5" params="name collider:=convex">
+        <xacro:property name="prefix" value="${name + '_' if name else ''}"/>
+        <link name="${prefix}base_link">
+            <inertial>
+                <origin xyz="-8.0961E-06 0.0019103 0.028995"/>
+                <mass value="0.90882"/>
+                <inertia ixx="0.0014545" ixy="4.2968E-08" ixz="-1.8199E-07" iyy="0.001345" iyz="-6.243E-06"
+                         izz="0.002155"/>
+            </inertial>
+            <visual>
+                <geometry>
+                    <mesh filename="file://$(find cr5_description)/meshes/visual/base_link.obj"/>
+                </geometry>
+            </visual>
+            <xacro:if value="${collider == 'convex'}">
+                <collision>
+                    <geometry>
+                        <mesh filename="file://$(find cr5_description)/meshes/collision/base_link.stl"/>
+                    </geometry>
+                </collision>
+            </xacro:if>
+            <xacro:if value="${collider == 'simple'}">
+                <collision>
+                    <origin xyz="0 0 0.05"/>
+                    <geometry>
+                        <cylinder length="0.1" radius="0.1"/>
+                    </geometry>
+                </collision>
+                <xacro:if value="${prefix == ''}">
+                    <collision>
+                        <origin xyz="0 0 -0.025"/>
+                        <geometry>
+                            <box size="1.5 1.5 0.05"/>
+                        </geometry>
+                    </collision>
+                </xacro:if>
+            </xacro:if>
+        </link>
+        <link name="${prefix}Link1">
+            <inertial>
+                <origin xyz="-8.7268E-07 -0.0032576 -0.0076748"/>
+                <mass value="1.6123"/>
+                <inertia ixx="0.0029122" ixy="5.7387E-09" ixz="1.9945E-08" iyy="0.0028191" iyz="0.00044094"
+                         izz="0.0032836"/>
+            </inertial>
+            <visual>
+                <geometry>
+                    <mesh filename="file://$(find cr5_description)/meshes/visual/Link1.obj"/>
+                </geometry>
+            </visual>
+            <xacro:if value="${collider == 'convex'}">
+                <collision>
+                    <geometry>
+                        <mesh filename="file://$(find cr5_description)/meshes/collision/Link1_0.stl"/>
+                    </geometry>
+                </collision>
+                <collision>
+                    <geometry>
+                        <mesh filename="file://$(find cr5_description)/meshes/collision/Link1_1.stl"/>
+                    </geometry>
+                </collision>
+            </xacro:if>
+            <xacro:if value="${collider == 'simple'}">
+                <collision>
+                    <geometry>
+                        <cylinder length="0.17" radius="0.08"/>
+                    </geometry>
+                </collision>
+            </xacro:if>
+        </link>
+        <joint name="${prefix}joint1" type="revolute">
+            <origin xyz="0 0 0.147"/>
+            <parent link="${prefix}base_link"/>
+            <child link="${prefix}Link1"/>
+            <axis xyz="0 0 1"/>
+            <limit lower="${-2*PI}" upper="${2*PI}" effort="300" velocity="${PI}"/>
+        </joint>
+        <link name="${prefix}Link2">
+            <inertial>
+                <origin xyz="-0.21351 -1.3842E-06 0.14252"/>
+                <mass value="5.5186"/>
+                <inertia ixx="0.0085919" ixy="7.5552E-07" ixz="-7.8922E-07" iyy="0.027553" iyz="1.4629E-07"
+                         izz="0.028294"/>
+            </inertial>
+            <visual>
+                <geometry>
+                    <mesh filename="file://$(find cr5_description)/meshes/visual/Link2.obj"/>
+                </geometry>
+            </visual>
+            <xacro:if value="${collider == 'convex'}">
+                <collision>
+                    <geometry>
+                        <mesh filename="file://$(find cr5_description)/meshes/collision/Link2_0.stl"/>
+                    </geometry>
+                </collision>
+                <collision>
+                    <geometry>
+                        <mesh filename="file://$(find cr5_description)/meshes/collision/Link2_1.stl"/>
+                    </geometry>
+                </collision>
+                <collision>
+                    <geometry>
+                        <mesh filename="file://$(find cr5_description)/meshes/collision/Link2_2.stl"/>
+                    </geometry>
+                </collision>
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
File: cr5_description/xacro/grippers.xacro (robot description, xacro)
@@ -17,5 +17,5 @@
 			<parent link="Link6"/>
 			<child link="flange"/>
-			<origin rpy="0 0 ${PI/2}"/>
+			<origin rpy="0 0 ${-PI/2}"/>
 		</joint>
 	</xacro:if>
@@ -37,3 +37,24 @@
 		</joint>
 	</xacro:if>
+	<xacro:if value="${'$(arg type)' == 'ft-90c'}">
+		<xacro:include filename="$(find changingtek_description)/xacro/AG2F90-C.xacro"/>
+		<link name="ft_sensor">
+			<visual>
+				<geometry>
+					<mesh filename="file://$(find cr5_description)/meshes/visual/ft_sensor.obj"/>
+				</geometry>
+			</visual>
+		</link>
+		<joint name="ft_sensor_joint" type="fixed">
+			<origin rpy="0 0 ${PI}"/>
+			<parent link="Link6"/>
+			<child link="ft_sensor"/>
+		</joint>
+		<xacro:AG2F90-C name="" use_flange="true"/>
+		<joint name="gripper_fix" type="fixed">
+			<parent link="ft_sensor"/>
+			<child link="flange"/>
+			<origin xyz="0 0 0.037" rpy="0 0 ${-PI/2}"/>
+		</joint>
+	</xacro:if>
 </robot>

File: cr5_description/xacro/ros2_control/robot.xacro (robot description, xacro)
@@ -27,9 +27,10 @@
       <xacro:if value="${'$(arg ros2_control_hardware_type)' == 'real'}">
         <plugin>dobot_ros2_control/DobotHardware</plugin>
-        <param name="robot_ip">192.168.5.38</param>
-        <param name="gain">800</param>
-        <param name="aheadtime">50</param>
-        <param name="speed_factor">100</param>
+        <param name="robot_ip">192.168.5.33</param>
+        <param name="gain">500</param>
+        <param name="aheadtime">20</param>
+        <param name="speed_factor">20</param>
         <param name="servo_time">0.05</param>
+        <param name="gripper_read_frequency_divider">50</param>
       </xacro:if>
     </hardware>
@@ -38,5 +39,5 @@
     <xacro:if value="${'$(arg ros2_control_hardware_type)' == 'real'}">
       <!-- 真实硬件模式：使用简单的gripper joint，仅有位置接口 -->
-      <xacro:if value="${'$(arg type)' == 'AG2F90-C-Soft'}">
+      <xacro:if value="${'$(arg type)' != 'empty'}">
         <joint name="gripper_joint">
           <command_interface name="position"/>
@@ -46,4 +47,13 @@
         </joint>
       </xacro:if>
+      <!-- 六维力传感器定义 -->
+      <sensor name="ft_sensor">
+        <state_interface name="force_x"/>
+        <state_interface name="force_y"/>
+        <state_interface name="force_z"/>
+        <state_interface name="torque_x"/>
+        <state_interface name="torque_y"/>
+        <state_interface name="torque_z"/>
+      </sensor>
     </xacro:if>
     <xacro:unless value="${'$(arg ros2_control_hardware_type)' == 'real'}">

File: cr5_dual_description/xacro/grippers.xacro (robot description, xacro)
@@ -51,7 +51,7 @@
     <xacro:AG2F90-C name="right" use_flange="true"/>
     <joint name="left_gripper_fixed" type="fixed">
-      <parent link="left_Link6"/>
+      <parent link="left_ft_sensor"/>
       <child link="left_flange"/>
-      <origin rpy="0 0 ${PI/2}"/>
+      <origin rpy="0 0 ${-PI/2}"/>
     </joint>
     <joint name="right_gripper_fixed" type="fixed">

File: cr5_dual_description/xacro/ros2_control/robot.xacro (robot description, xacro)
@@ -15,8 +15,9 @@
                 <plugin>dobot_ros2_control/DobotHardware</plugin>
                 <param name="robot_ip">192.168.5.33</param>
-                <param name="gain">200</param>
+                <param name="gain">500</param>
                 <param name="aheadtime">20</param>
-                <param name="speed_factor">100</param>
-                <param name="servo_time">0.3</param>
+                <param name="speed_factor">20</param>
+                <param name="servo_time">0.05</param>
+                <param name="gripper_read_frequency_divider">50</param>
             </hardware>
             <xacro:cr5_interfaces name="left"/>
@@ -29,24 +30,34 @@
                 </joint>
             </xacro:if>
+            <sensor name="left_ft_sensor">
+                <state_interface name="force_x"/>
+                <state_interface name="force_y"/>
+                <state_interface name="force_z"/>
+                <state_interface name="torque_x"/>
+                <state_interface name="torque_y"/>
+                <state_interface name="torque_z"/>
+            </sensor>
         </ros2_control>
-        <ros2_control name="cr5_right_system" type="system">
-            <hardware>
-                <plugin>dobot_ros2_control/DobotHardware</plugin>
-                <param name="robot_ip">192.168.5.34</param>
-                <param name="gain">200</param>
-                <param name="aheadtime">20</param>
-                <param name="speed_factor">100</param>
-                <param name="servo_time">0.3</param>
-            </hardware>
-            <xacro:cr5_interfaces name="right"/>
-            <xacro:if value="${'$(arg type)' != 'empty'}">
-                <joint name="right_gripper_joint">
-                    <command_interface name="position"/>
-                    <state_interface name="position">
-                        <param name="initial_value">0</param>
-                    </state_interface>
-                </joint>
-            </xacro:if>
-        </ros2_control>
+        <xacro:unless value="${'$(arg type)' == 'left_arm'}">
+            <ros2_control name="cr5_right_system" type="system">
+                <hardware>
+                    <plugin>dobot_ros2_control/DobotHardware</plugin>
+                    <param name="robot_ip">192.168.5.34</param>
+                    <param name="gain">200</param>
+                    <param name="aheadtime">20</param>
+                    <param name="speed_factor">100</param>
+                    <param name="servo_time">0.3</param>
+                </hardware>
+                <xacro:cr5_interfaces name="right"/>
+                <xacro:if value="${'$(arg type)' != 'empty'}">
+                    <joint name="right_gripper_joint">
+                        <command_interface name="position"/>
+                        <state_interface name="position">
+                            <param name="initial_value">0</param>
+                        </state_interface>
+                    </joint>
+                </xacro:if>
+            </ros2_control>
+        </xacro:unless>
     </xacro:if>
     <xacro:if value="${'$(arg ros2_control_hardware_type)' == 'isaac'}">
@@ -147,5 +158,6 @@
             <xacro:cr5_interfaces name="right"/>
             <!-- 夹爪接口 - 参考CR5的模块化设计 -->
-            <xacro:if value="${'$(arg type)' == 'AG2F90-C' or '$(arg type)' == 'AG2F90-C-Soft'  or '$(arg type)' == 'left_arm'}">
+            <xacro:if
+                    value="${'$(arg type)' == 'AG2F90-C' or '$(arg type)' == 'AG2F90-C-Soft'  or '$(arg type)' == 'left_arm'}">
                 <xacro:include filename="$(find changingtek_description)/xacro/ros2_control/AG2F90-C.xacro"/>
                 <xacro:ag2f90c_interfaces name="left"/>

Commit message: add ft 90c ocs2 control config

File: cr5_description/xacro/arm.xacro (robot description, xacro)
@@ -226,5 +226,5 @@
             <child link="${prefix}Link4"/>
             <axis xyz="0 0 1"/>
-            <limit lower="${-2*PI}" upper="2.2591366109921265" effort="300" velocity="${PI}"/>
+            <limit lower="${-2*PI}" upper="${2*PI}" effort="300" velocity="${PI}"/>
         </joint>
         <link name="${prefix}Link5">
