Commit message: add dh param

File: cr5_description/xacro/arm.xacro (robot description, xacro)
@@ -2,5 +2,5 @@
 <robot name="cr5_robot" xmlns:xacro="http://ros.org/wiki/xacro">
 	<xacro:property name="PI" value="3.1415926535897931"/>
-	<xacro:macro name="CR5" params="name collider:=convex">
+	<xacro:macro name="CR5" params="name collider:=convex tf_params">
 		<xacro:property name="prefix" value="${name + '_' if name else ''}"/>
 		<link name="${prefix}base_link">
@@ -8,5 +8,5 @@
 				<origin xyz="-8.0961E-06 0.0019103 0.028995"/>
 				<mass value="0.90882"/>
-			<inertia ixx="0.0014545" ixy="4.2968E-08" ixz="-1.8199E-07" iyy="0.001345" iyz="-6.243E-06" izz="0.002155"/>
+				<inertia ixx="0.0014545" ixy="4.2968E-08" ixz="-1.8199E-07" iyy="0.001345" iyz="-6.243E-06" izz="0.002155"/>
 			</inertial>
 			<visual>
@@ -43,5 +43,5 @@
 				<origin xyz="-8.7268E-07 -0.0032576 -0.0076748"/>
 				<mass value="1.6123"/>
-			<inertia ixx="0.0029122" ixy="5.7387E-09" ixz="1.9945E-08" iyy="0.0028191" iyz="0.00044094" izz="0.0032836"/>
+				<inertia ixx="0.0029122" ixy="5.7387E-09" ixz="1.9945E-08" iyy="0.0028191" iyz="0.00044094" izz="0.0032836"/>
 			</inertial>
 			<visual>
@@ -70,8 +70,8 @@
 			</xacro:if>
 		</link>
-	<joint name="${prefix}joint1" type="revolute">
-		<origin xyz="0 0 0.147"/>
-		<parent link="${prefix}base_link"/>
-		<child link="${prefix}Link1"/>
+		<joint name="${prefix}joint1" type="revolute">
+			<origin xyz="${tf_params['joint1']['xyz']}" rpy="${tf_params['joint1']['rpy']}"/>
+			<parent link="${prefix}base_link"/>
+			<child link="${prefix}Link1"/>
 			<axis xyz="0 0 1"/>
 			<limit lower="${-2*PI}" upper="${2*PI}" effort="300" velocity="${PI}"/>
@@ -81,5 +81,5 @@
 				<origin xyz="-0.21351 -1.3842E-06 0.14252"/>
 				<mass value="5.5186"/>
-			<inertia ixx="0.0085919" ixy="7.5552E-07" ixz="-7.8922E-07" iyy="0.027553" iyz="1.4629E-07" izz="0.028294"/>
+				<inertia ixx="0.0085919" ixy="7.5552E-07" ixz="-7.8922E-07" iyy="0.027553" iyz="1.4629E-07" izz="0.028294"/>
 			</inertial>
 			<visual>
@@ -126,8 +126,8 @@
 			</xacro:if>
 		</link>
-	<joint name="${prefix}joint2" type="revolute">
-		<origin rpy="${PI/2} ${PI/2} 0"/>
-		<parent link="${prefix}Link1"/>
-		<child link="${prefix}Link2"/>
+		<joint name="${prefix}joint2" type="revolute">
+			<origin xyz="${tf_params['joint2']['xyz']}" rpy="${tf_params['joint2']['rpy']}"/>
+			<parent link="${prefix}Link1"/>
+			<child link="${prefix}Link2"/>
 			<axis xyz="0 0 1"/>
 			<limit lower="${-2*PI}" upper="${2*PI}" effort="300" velocity="${PI}"/>
@@ -137,5 +137,5 @@
 				<origin xyz="-0.15231 -1.4079E-07 0.022693"/>
 				<mass value="2.8536"/>
-			<inertia ixx="0.0032608" ixy="-3.2147E-10" ixz="0.00012363" iyy="0.0092967" iyz="2.9478E-10" izz="0.0095552"/>
+				<inertia ixx="0.0032608" ixy="-3.2147E-10" ixz="0.00012363" iyy="0.0092967" iyz="2.9478E-10" izz="0.0095552"/>
 			</inertial>
 			<visual>
@@ -182,8 +182,8 @@
 			</xacro:if>
 		</link>
-	<joint name="${prefix}joint3" type="revolute">
-		<origin xyz="-0.427 0 0"/>
-		<parent link="${prefix}Link2"/>
-		<child link="${prefix}Link3"/>
+		<joint name="${prefix}joint3" type="revolute">
+			<origin xyz="${tf_params['joint3']['xyz']}" rpy="${tf_params['joint3']['rpy']}"/>
+			<parent link="${prefix}Link2"/>
+			<child link="${prefix}Link3"/>
 			<axis xyz="0 0 1"/>
 			<limit lower="-2.7925" upper="2.7925" effort="300" velocity="3.14159"/>
@@ -193,5 +193,6 @@
 				<origin xyz="-3.2386E-07 -0.002077 -0.0015548"/>
 				<mass value="0.67058"/>
-			<inertia ixx="0.00066939" ixy="4.1975E-10" ixz="-1.0734E-08" iyy="0.00065424" iyz="0.00011081" izz="0.00065365"/>
+				<inertia ixx="0.00066939" ixy="4.1975E-10" ixz="-1.0734E-08" iyy="0.00065424" iyz="0.00011081"
+								 izz="0.00065365"/>
 			</inertial>
 			<visual>
@@ -216,8 +217,8 @@
 			</xacro:if>
 		</link>
-	<joint name="${prefix}joint4" type="revolute">
-		<origin xyz="-0.357 0 0.141" rpy="0 0 ${-PI/2}"/>
-		<parent link="${prefix}Link3"/>
-		<child link="${prefix}Link4"/>
+		<joint name="${prefix}joint4" type="revolute">
+			<origin xyz="${tf_params['joint4']['xyz']}" rpy="${tf_params['joint4']['rpy']}"/>
+			<parent link="${prefix}Link3"/>
+			<child link="${prefix}Link4"/>
 			<axis xyz="0 0 1"/>
 			<limit lower="${-2*PI}" upper="${2*PI}" effort="300" velocity="${PI}"/>
@@ -227,5 +228,6 @@
 				<origin xyz="-3.7738E-07 -0.0045777 -0.0012971"/>
 				<mass value="0.7269"/>
-			<inertia ixx="0.00073069" ixy="-5.7806E-09" ixz="6.7132E-09" iyy="0.00071195" iyz="-0.00011926" izz="0.00071391"/>
+				<inertia ixx="0.00073069" ixy="-5.7806E-09" ixz="6.7132E-09" iyy="0.00071195" iyz="-0.00011926"
+								 izz="0.00071391"/>
 			</inertial>
 			<visual>
@@ -250,8 +252,8 @@
 			</xacro:if>
 		</link>
-	<joint name="${prefix}joint5" type="revolute">
-		<origin xyz="0 -0.116 0" rpy="${PI/2} 0 0"/>
-		<parent link="${prefix}Link4"/>
-		<child link="${prefix}Link5"/>
+		<joint name="${prefix}joint5" type="revolute">
+			<origin xyz="${tf_params['joint5']['xyz']}" rpy="${tf_params['joint5']['rpy']}"/>
+			<parent link="${prefix}Link4"/>
+			<child link="${prefix}Link5"/>
 			<axis xyz="0 0 1"/>
 			<limit lower="${-2*PI}" upper="${2*PI}" effort="300" velocity="${PI}"/>
@@ -261,5 +263,6 @@
 				<origin xyz="5.0777E-11 9.3774E-05 -0.019285"/>
 				<mass value="0.15789"/>
-			<inertia ixx="7.8045E-05" ixy="6.1582E-15" ixz="6.2471E-14" iyy="7.9168E-05" iyz="-1.3822E-07" izz="0.00012951"/>
+				<inertia ixx="7.8045E-05" ixy="6.1582E-15" ixz="6.2471E-14" iyy="7.9168E-05" iyz="-1.3822E-07"
+								 izz="0.00012951"/>
 			</inertial>
 			<visual>
@@ -284,8 +287,8 @@
 			</xacro:if>
 		</link>
-	<joint name="${prefix}joint6" type="revolute">
-		<origin xyz="0 0.105 0" rpy="${-PI/2} 0 0"/>
-		<parent link="${prefix}Link5"/>
-		<child link="${prefix}Link6"/>
+		<joint name="${prefix}joint6" type="revolute">
+			<origin xyz="${tf_params['joint6']['xyz']}" rpy="${tf_params['joint6']['rpy']}"/>
+			<parent link="${prefix}Link5"/>
+			<child link="${prefix}Link6"/>
 			<axis xyz="0 0 1"/>
 			<limit lower="${-2*PI}" upper="${2*PI}" effort="300" velocity="${PI}"/>

File: cr5_description/xacro/robot.xacro (robot description, xacro)
@@ -2,6 +2,8 @@
 <robot name="DobotCR5" xmlns:xacro="http://www.ros.org/wiki/xacro">
   <xacro:arg name="collider" default="convex"/>
+  <!-- 从同目录下的tf_params.yaml文件加载tf参数 -->
+  <xacro:property name="tf_params" value="${xacro.load_yaml('$(find cr5_description)/xacro/tf_params.yaml')['tf_params']}"/>
   <xacro:include filename="$(find cr5_description)/xacro/arm.xacro"/>
-  <xacro:CR5 name="" collider="$(arg collider)"/>
+  <xacro:CR5 name="" collider="$(arg collider)" tf_params="${tf_params}"/>
   <xacro:include filename="$(find cr5_description)/xacro/grippers.xacro"/>
 </robot>

Commit message: fix dh param

File: cr5_description/xacro/arm.xacro (robot description, xacro)
@@ -2,6 +2,56 @@
 <robot name="cr5_robot" xmlns:xacro="http://ros.org/wiki/xacro">
     <xacro:property name="PI" value="3.1415926535897931"/>
-    <xacro:macro name="CR5" params="name collider:=convex tf_params">
+    <xacro:property name="DEG2RAD" value="0.017453292519943295"/>  <!-- PI/180 -->
+    <xacro:property name="MM2M" value="0.001"/>  <!-- 毫米转米 -->
+    <xacro:macro name="CR5" params="name collider:=convex dh_params">
         <xacro:property name="prefix" value="${name + '_' if name else ''}"/>
+        <!--
+            从DH参数计算各关节的xyz和rpy值（单位转换：毫米->米，度->弧度）
+            标准DH参数映射规则（基于执行器轴方向）：
+            - a (link length): 沿着x轴的距离 → xyz的x分量
+            - d (link offset): 沿着z轴的距离 → xyz的z分量
+            - alpha (twist): 绕x轴的旋转角度 → rpy的x分量（roll）
+            - theta: 绕z轴的旋转（关节变量，在URDF中通过axis定义）
+        -->
+        <!-- joint1: 标准DH转换 - a=0, d=147mm, alpha=0 -->
+        <xacro:property name="j1_a_m" value="${dh_params['joint1']['a'] * MM2M}"/>
+        <xacro:property name="j1_d_m" value="${dh_params['joint1']['d'] * MM2M}"/>
+        <xacro:property name="j1_alpha_rad" value="${dh_params['joint1']['alpha'] * DEG2RAD}"/>
+        <xacro:property name="j1_xyz" value="${str(j1_a_m) + ' ' + str(0) + ' ' + str(j1_d_m)}"/>
+        <xacro:property name="j1_rpy" value="${str(j1_alpha_rad) + ' ' + str(0) + ' ' + str(0)}"/>
+        <!-- joint2: alpha映射到rpy的x（roll），theta的固定偏移π/2映射到rpy的y（pitch） -->
+        <xacro:property name="j2_a_m" value="${dh_params['joint2']['a'] * MM2M}"/>
+        <xacro:property name="j2_d_m" value="${dh_params['joint2']['d'] * MM2M}"/>
+        <xacro:property name="j2_alpha_rad" value="${dh_params['joint2']['alpha'] * DEG2RAD}"/>
+        <xacro:property name="j2_xyz" value="${str(j2_a_m) + ' ' + str(0) + ' ' + str(j2_d_m)}"/>
+        <!-- alpha -> rpy x (roll), theta的固定偏移π/2 -> rpy y (pitch) -->
+        <xacro:property name="j2_rpy" value="${str(j2_alpha_rad) + ' ' + str(PI/2) + ' ' + str(0)}"/>
+        <!-- joint3: 标准DH转换 - a=-427.567mm, d=0, alpha≈0 -->
+        <xacro:property name="j3_a_m" value="${dh_params['joint3']['a'] * MM2M}"/>
+        <xacro:property name="j3_d_m" value="${dh_params['joint3']['d'] * MM2M}"/>
+        <xacro:property name="j3_alpha_rad" value="${dh_params['joint3']['alpha'] * DEG2RAD}"/>
+        <xacro:property name="j3_xyz" value="${str(j3_a_m) + ' ' + str(0) + ' ' + str(j3_d_m)}"/>
+        <xacro:property name="j3_rpy" value="${str(j3_alpha_rad) + ' ' + str(0) + ' ' + str(0)}"/>
+        <!-- joint4: alpha映射到rpy的x（roll），theta的固定偏移-π/2映射到rpy的z（yaw） -->
+        <xacro:property name="j4_a_m" value="${dh_params['joint4']['a'] * MM2M}"/>
+        <xacro:property name="j4_d_m" value="${dh_params['joint4']['d'] * MM2M}"/>
+        <xacro:property name="j4_alpha_rad" value="${dh_params['joint4']['alpha'] * DEG2RAD}"/>
+        <xacro:property name="j4_xyz" value="${str(j4_a_m) + ' ' + str(0) + ' ' + str(j4_d_m)}"/>
+        <!-- alpha -> rpy x (roll), theta的固定偏移-π/2 -> rpy z (yaw) -->
+        <xacro:property name="j4_rpy" value="${str(j4_alpha_rad) + ' ' + str(0) + ' ' + str(-PI/2)}"/>
+        <!-- joint5: 由于坐标系旋转，d映射到y负方向，alpha仍为roll -->
+        <xacro:property name="j5_a_m" value="${dh_params['joint5']['a'] * MM2M}"/>
+        <xacro:property name="j5_d_m" value="${dh_params['joint5']['d'] * MM2M}"/>
+        <xacro:property name="j5_alpha_rad" value="${dh_params['joint5']['alpha'] * DEG2RAD}"/>
+        <!-- 注意：由于坐标系旋转，d映射到y负方向而不是z方向 -->
+        <xacro:property name="j5_xyz" value="${str(j5_a_m) + ' ' + str(-j5_d_m) + ' ' + str(0)}"/>
+        <xacro:property name="j5_rpy" value="${str(j5_alpha_rad) + ' ' + str(0) + ' ' + str(0)}"/>
+        <!-- joint6: 由于坐标系旋转，d映射到y正方向，alpha仍为roll -->
+        <xacro:property name="j6_a_m" value="${dh_params['joint6']['a'] * MM2M}"/>
+        <xacro:property name="j6_d_m" value="${dh_params['joint6']['d'] * MM2M}"/>
+        <xacro:property name="j6_alpha_rad" value="${dh_params['joint6']['alpha'] * DEG2RAD}"/>
+        <!-- 注意：由于坐标系旋转，d映射到y正方向而不是z方向 -->
+        <xacro:property name="j6_xyz" value="${str(j6_a_m) + ' ' + str(j6_d_m) + ' ' + str(0)}"/>
+        <xacro:property name="j6_rpy" value="${str(j6_alpha_rad) + ' ' + str(0) + ' ' + str(0)}"/>
         <link name="${prefix}base_link">
             <inertial>
@@ -73,5 +123,5 @@
         </link>
         <joint name="${prefix}joint1" type="revolute">
-            <origin xyz="${tf_params['joint1']['xyz']}" rpy="${tf_params['joint1']['rpy']}"/>
+            <origin xyz="${j1_xyz}" rpy="${j1_rpy}"/>
             <parent link="${prefix}base_link"/>
             <child link="${prefix}Link1"/>
@@ -130,5 +180,5 @@
         </link>
         <joint name="${prefix}joint2" type="revolute">
-            <origin xyz="${tf_params['joint2']['xyz']}" rpy="${tf_params['joint2']['rpy']}"/>
+            <origin xyz="${j2_xyz}" rpy="${j2_rpy}"/>
             <parent link="${prefix}Link1"/>
             <child link="${prefix}Link2"/>
@@ -187,5 +237,5 @@
         </link>
         <joint name="${prefix}joint3" type="revolute">
-            <origin xyz="${tf_params['joint3']['xyz']}" rpy="${tf_params['joint3']['rpy']}"/>
+            <origin xyz="${j3_xyz}" rpy="${j3_rpy}"/>
             <parent link="${prefix}Link2"/>
             <child link="${prefix}Link3"/>
@@ -222,5 +272,5 @@
         </link>
         <joint name="${prefix}joint4" type="revolute">
-            <origin xyz="${tf_params['joint4']['xyz']}" rpy="${tf_params['joint4']['rpy']}"/>
+            <origin xyz="${j4_xyz}" rpy="${j4_rpy}"/>
             <parent link="${prefix}Link3"/>
             <child link="${prefix}Link4"/>
@@ -257,5 +307,5 @@
         </link>
         <joint name="${prefix}joint5" type="revolute">
-            <origin xyz="${tf_params['joint5']['xyz']}" rpy="${tf_params['joint5']['rpy']}"/>
+            <origin xyz="${j5_xyz}" rpy="${j5_rpy}"/>
             <parent link="${prefix}Link4"/>
             <child link="${prefix}Link5"/>
@@ -292,5 +342,5 @@
         </link>
         <joint name="${prefix}joint6" type="revolute">
-            <origin xyz="${tf_params['joint6']['xyz']}" rpy="${tf_params['joint6']['rpy']}"/>
+            <origin xyz="${j6_xyz}" rpy="${j6_rpy}"/>
             <parent link="${prefix}Link5"/>
             <child link="${prefix}Link6"/>

File: cr5_description/xacro/robot.xacro (robot description, xacro)
@@ -2,8 +2,8 @@
 <robot name="DobotCR5" xmlns:xacro="http://www.ros.org/wiki/xacro">
   <xacro:arg name="collider" default="convex"/>
-  <!-- 从同目录下的tf_params.yaml文件加载tf参数 -->
-  <xacro:property name="tf_params" value="${xacro.load_yaml('$(find cr5_description)/xacro/tf_params.yaml')['tf_params']}"/>
+  <!-- 从同目录下的dh_params.yaml文件加载DH参数 -->
+  <xacro:property name="dh_params" value="${xacro.load_yaml('$(find cr5_description)/xacro/dh_params.yaml')['dh_params']}"/>
   <xacro:include filename="$(find cr5_description)/xacro/arm.xacro"/>
-  <xacro:CR5 name="" collider="$(arg collider)" tf_params="${tf_params}"/>
+  <xacro:CR5 name="" collider="$(arg collider)" dh_params="${dh_params}"/>
   <xacro:include filename="$(find cr5_description)/xacro/grippers.xacro"/>
 </robot>

File: cr5_description/xacro/ros2_control/robot.xacro (robot description, xacro)
@@ -1,83 +1,85 @@
 <?xml version="1.0"?>
 <robot xmlns:xacro="http://www.ros.org/wiki/xacro" name="CR5">
-  <xacro:arg name="ros2_control_hardware_type" default="mock_components"/>
-  <link name="world"/>
-  <joint name="world_fixed" type="fixed">
-    <parent link="world"/>
-    <child link="base_link"/>
-    <origin/>
-  </joint>
-  <xacro:include filename="$(find cr5_description)/xacro/robot.xacro"/>
-  <xacro:include filename="$(find cr5_description)/xacro/ros2_control/interfaces.xacro"/>
-  <ros2_control name="cr5System" type="system">
-    <hardware>
-      <xacro:if value="${'$(arg ros2_control_hardware_type)' == 'gz'}">
-        <plugin>gz_ros2_control/GazeboSimSystem</plugin>
-      </xacro:if>
-      <xacro:if value="${'$(arg ros2_control_hardware_type)' == 'mock_components'}">
-        <plugin>mock_components/GenericSystem</plugin>
-      </xacro:if>
-      <xacro:if value="${'$(arg ros2_control_hardware_type)' == 'isaac'}">
-        <plugin>topic_based_ros2_control/TopicBasedSystem</plugin>
-        <param name="joint_commands_topic">/isaac/joint_command</param>
-        <param name="joint_states_topic">/isaac/joint_states</param>
-        <param name="sum_wrapped_joint_states">false</param>
-        <param name="initialize_commands_from_state">true</param>
-      </xacro:if>
-      <xacro:if value="${'$(arg ros2_control_hardware_type)' == 'real'}">
-        <plugin>dobot_ros2_control/DobotHardware</plugin>
-        <param name="robot_ip">192.168.5.33</param>
-        <param name="gain">500</param>
-        <param name="aheadtime">20</param>
-        <param name="speed_factor">1</param>
-        <param name="servo_time">0.02</param>
-        <param name="gripper_read_frequency_divider">50</param>
-      </xacro:if>
-    </hardware>
-    <xacro:cr5_interfaces name=""/>
-    <!-- 夹爪接口定义 -->
-    <xacro:if value="${'$(arg ros2_control_hardware_type)' == 'real'}">
-      <!-- 真实硬件模式：使用简单的gripper joint，仅有位置接口 -->
-      <xacro:if value="${'$(arg type)' != 'empty'}">
-        <joint name="gripper_joint">
-          <command_interface name="position"/>
-          <state_interface name="position">
-            <param name="initial_value">0</param>
-          </state_interface>
-        </joint>
-      </xacro:if>
-      <!-- 六维力传感器定义 -->
-      <sensor name="ft_sensor">
-        <state_interface name="force.x"/>
-        <state_interface name="force.y"/>
-        <state_interface name="force.z"/>
-        <state_interface name="torque.x"/>
-        <state_interface name="torque.y"/>
-        <state_interface name="torque.z"/>
-      </sensor>
+    <xacro:arg name="ros2_control_hardware_type" default="mock_components"/>
+    <link name="world"/>
+    <joint name="world_fixed" type="fixed">
+        <parent link="world"/>
+        <child link="base_link"/>
+        <origin/>
+    </joint>
+    <xacro:include filename="$(find cr5_description)/xacro/robot.xacro"/>
+    <xacro:include filename="$(find cr5_description)/xacro/ros2_control/interfaces.xacro"/>
+    <ros2_control name="cr5System" type="system">
+        <hardware>
+            <xacro:if value="${'$(arg ros2_control_hardware_type)' == 'gz'}">
+                <plugin>gz_ros2_control/GazeboSimSystem</plugin>
+            </xacro:if>
+            <xacro:if value="${'$(arg ros2_control_hardware_type)' == 'mock_components'}">
+                <plugin>mock_components/GenericSystem</plugin>
+            </xacro:if>
+            <xacro:if value="${'$(arg ros2_control_hardware_type)' == 'isaac'}">
+                <plugin>topic_based_ros2_control/TopicBasedSystem</plugin>
+                <param name="joint_commands_topic">/isaac/joint_command</param>
+                <param name="joint_states_topic">/isaac/joint_states</param>
+                <param name="sum_wrapped_joint_states">false</param>
+                <param name="initialize_commands_from_state">true</param>
+            </xacro:if>
+            <xacro:if value="${'$(arg ros2_control_hardware_type)' == 'real'}">
+                <plugin>dobot_ros2_control/DobotHardware</plugin>
+                <param name="robot_ip">192.168.5.33</param>
+                <param name="gain">500</param>
+                <param name="aheadtime">20</param>
+                <param name="speed_factor">1</param>
+                <param name="servo_time">0.02</param>
+                <param name="gripper_read_frequency_divider">50</param>
+            </xacro:if>
+        </hardware>
+        <xacro:cr5_interfaces name=""/>
+        <!-- 夹爪接口定义 -->
+        <xacro:if value="${'$(arg ros2_control_hardware_type)' == 'real'}">
+            <!-- 真实硬件模式：使用简单的gripper joint，仅有位置接口 -->
+            <xacro:if value="${'$(arg type)' != 'empty'}">
+                <joint name="gripper_joint">
+                    <command_interface name="position"/>
+                    <state_interface name="position">
+                        <param name="initial_value">0</param>
+                    </state_interface>
+                </joint>
+            </xacro:if>
+            <xacro:if value="${'$(arg type)' == 'ft-90c'}">
+                <!-- 六维力传感器定义 -->
+                <sensor name="ft_sensor">
+                    <state_interface name="force.x"/>
+                    <state_interface name="force.y"/>
+                    <state_interface name="force.z"/>
+                    <state_interface name="torque.x"/>
+                    <state_interface name="torque.y"/>
+                    <state_interface name="torque.z"/>
+                </sensor>
+            </xacro:if>
+        </xacro:if>
+        <xacro:unless value="${'$(arg ros2_control_hardware_type)' == 'real'}">
+            <!-- 非真实硬件模式：使用现有的夹爪定义 -->
+            <xacro:if value="${'$(arg type)' == 'AG2F90-C' or '$(arg type)' == 'AG2F90-C-Soft'}">
+                <xacro:include filename="$(find changingtek_description)/xacro/ros2_control/AG2F90-C.xacro"/>
+                <xacro:ag2f90c_interfaces name=""/>
+            </xacro:if>
+            <xacro:if value="${'$(arg type)' == 'AG2F120S'}">
+                <xacro:include filename="$(find changingtek_description)/xacro/ros2_control/AG2F120S.xacro"/>
+                <xacro:ag2f120s_interfaces name=""/>
+            </xacro:if>
+            <xacro:if value="${'$(arg type)' == 'robotiq85'}">
+                <xacro:include filename="$(find robotiq_description)/xacro/ros2_control/2F85.xacro"/>
+                <xacro:robotiq_2f85_interfaces name=""/>
+            </xacro:if>
+        </xacro:unless>
+    </ros2_control>
+    <xacro:arg name="gazebo" default="false"/>
+    <xacro:if value="$(arg gazebo)">
+        <gazebo>
+            <plugin filename="gz_ros2_control-system" name="gz_ros2_control::GazeboSimROS2ControlPlugin">
+                <parameters>$(find cr5_description)/config/ros2_control/ros2_controllers.yaml</parameters>
+            </plugin>
+        </gazebo>
     </xacro:if>
-    <xacro:unless value="${'$(arg ros2_control_hardware_type)' == 'real'}">
-      <!-- 非真实硬件模式：使用现有的夹爪定义 -->
-      <xacro:if value="${'$(arg type)' == 'AG2F90-C' or '$(arg type)' == 'AG2F90-C-Soft'}">
-        <xacro:include filename="$(find changingtek_description)/xacro/ros2_control/AG2F90-C.xacro"/>
-        <xacro:ag2f90c_interfaces name=""/>
-      </xacro:if>
-      <xacro:if value="${'$(arg type)' == 'AG2F120S'}">
-        <xacro:include filename="$(find changingtek_description)/xacro/ros2_control/AG2F120S.xacro"/>
-        <xacro:ag2f120s_interfaces name=""/>
-      </xacro:if>
-      <xacro:if value="${'$(arg type)' == 'robotiq85'}">
-        <xacro:include filename="$(find robotiq_description)/xacro/ros2_control/2F85.xacro"/>
-        <xacro:robotiq_2f85_interfaces name=""/>
-      </xacro:if>
-    </xacro:unless>
-  </ros2_control>
-  <xacro:arg name="gazebo" default="false"/>
-  <xacro:if value="$(arg gazebo)">
-    <gazebo>
-      <plugin filename="gz_ros2_control-system" name="gz_ros2_control::GazeboSimROS2ControlPlugin">
-        <parameters>$(find cr5_description)/config/ros2_control/ros2_controllers.yaml</parameters>
-      </plugin>
-    </gazebo>
-  </xacro:if>
 </robot>
