Commit message: fix cr5 config

File: cr5_description/xacro/arm.xacro (robot description, xacro)
@@ -23,10 +23,4 @@
 			</xacro:if>
 			<xacro:if value="${collider == 'simple'}">
-				<collision>
-					<origin xyz="0 0 0.05"/>
-					<geometry>
-						<cylinder length="0.1" radius="0.1"/>
-					</geometry>
-				</collision>
 				<xacro:if value="${prefix == ''}">
 					<collision>

File: cr5_description/xacro/grippers.xacro (robot description, xacro)
@@ -5,17 +5,37 @@
 	  - selected_gripper_type: empty / robotiq85 / AG2F90-C(-Soft) / AG2F120S ...
 	  - selected_scene: 可选（当前文件不使用）
+	  OCS2 planning URDF: eef_fixed_joints:=true 时冻结夹爪驱动关节（见 robot_common_launch planning mappings）。
 	-->
+	<xacro:property name="eef_fixed" value="$(arg eef_fixed_joints)"/>
+	<xacro:property name="kinematic_only" value="${str(eef_fixed).lower() == 'true'}"/>
+	<!-- 无夹爪：planning 需要在 Link6 上提供 OCS2 eeFrame -->
+	<xacro:if value="${selected_gripper_type == 'empty' and kinematic_only}">
+		<link name="eef"/>
+		<joint name="eef_joint" type="fixed">
+			<parent link="Link6"/>
+			<child link="eef"/>
+		</joint>
+	</xacro:if>
 	<!-- 根据type参数决定使用哪种夹爪 -->
 	<xacro:if value="${selected_gripper_type == 'robotiq85'}">
-		<xacro:include filename="$(find robotiq_description)/xacro/2F85.xacro"/>
-		<xacro:Robotiq85 name=""/>
-		<joint name="gripper_fix" type="fixed">
-			<parent link="Link6"/>
-			<child link="gripper_base"/>
-		</joint>
+		<xacro:if value="${kinematic_only}">
+			<link name="eef"/>
+			<joint name="eef_joint" type="fixed">
+				<parent link="Link6"/>
+				<child link="eef"/>
+			</joint>
+		</xacro:if>
+		<xacro:unless value="${kinematic_only}">
+			<xacro:include filename="$(find robotiq_description)/xacro/2F85.xacro"/>
+			<xacro:Robotiq85 name=""/>
+			<joint name="gripper_fix" type="fixed">
+				<parent link="Link6"/>
+				<child link="gripper_base"/>
+			</joint>
+		</xacro:unless>
 	</xacro:if>
 	<xacro:if value="${selected_gripper_type == 'AG2F90-C'}">
 		<xacro:include filename="$(find changingtek_description)/xacro/AG2F90-C.xacro"/>
-		<xacro:AG2F90-C name="" use_flange="true"/>
+		<xacro:AG2F90-C name="" use_flange="true" kinematic_only="${kinematic_only}"/>
 		<joint name="gripper_fix" type="fixed">
 			<parent link="Link6"/>
@@ -26,5 +46,5 @@
 	<xacro:if value="${selected_gripper_type == 'AG2F90-C-Soft'}">
 		<xacro:include filename="$(find changingtek_description)/xacro/AG2F90-C.xacro"/>
-		<xacro:AG2F90-C name="" use_flange="true" pad="soft"/>
+		<xacro:AG2F90-C name="" use_flange="true" pad="soft" kinematic_only="${kinematic_only}"/>
 		<joint name="gripper_fix" type="fixed">
 			<parent link="Link6"/>
@@ -32,14 +52,16 @@
 			<origin rpy="0 0 ${PI/2}"/>
 		</joint>
-		<link name="hand_camera"/>
-		<joint name="hand_camera_joint" type="fixed">
-			<parent link="Link6"/>
-			<child link="hand_camera"/>
-			<origin xyz="-0.0232323851 -0.0658349999 0.1368881312" rpy="-0.1206332889 0.0085965555 0.0669556163"/>
-		</joint>
+		<xacro:unless value="${kinematic_only}">
+			<link name="hand_camera"/>
+			<joint name="hand_camera_joint" type="fixed">
+				<parent link="Link6"/>
+				<child link="hand_camera"/>
+				<origin xyz="-0.0232323851 -0.0658349999 0.1368881312" rpy="-0.1206332889 0.0085965555 0.0669556163"/>
+			</joint>
+		</xacro:unless>
 	</xacro:if>
 	<xacro:if value="${selected_gripper_type == 'AG2F120S'}">
 		<xacro:include filename="$(find changingtek_description)/xacro/AG2F120S.xacro"/>
-		<xacro:AG2F120S name=""/>
+		<xacro:AG2F120S name="" kinematic_only="${kinematic_only}"/>
 		<joint name="gripper_fix" type="fixed">
 			<parent link="Link6"/>

File: cr5_description/xacro/robot.xacro (robot description, xacro)
@@ -4,4 +4,6 @@
   <xacro:arg name="type" default="empty"/>
   <xacro:arg name="scene" default=""/>
+  <!-- false: ros2_control / 可视化；OCS2 planning 由 robot_common_launch 注入 eef_fixed_joints:=true -->
+  <xacro:arg name="eef_fixed_joints" default="false"/>
   <!--
     CR5 的 type 不仅用于末端夹爪，也可承载场景(scene)信息（类似 m6_ccs_description 的机制）。
