Commit message: fix dobot collision problem

File: cr5_description/xacro/arm.xacro (robot description, xacro)
@@ -272,12 +272,4 @@
 				</collision>
 			</xacro:if>
-			<xacro:if value="${collider == 'simple'}">
-				<collision>
-					<origin xyz="0 0 0.1"/>
-					<geometry>
-						<box size="0.05 0.15 0.2"/>
-					</geometry>
-				</collision>
-			</xacro:if>
 		</link>
 		<joint name="${prefix}joint6" type="revolute">
